File: isometric-75-pcb-iso/isometric-75-pcb-iso.kicad_pcb (KiCad board)
At the start: 2 copper layers, 308.8 x 123.5 mm, 314 parts, among them J101 USB, J102 SPI, J103 Conn_01x06_Male, Q101 AO3400A, SW101 RST, SW102 BOOT, SW201 Rotary_Encoder_Switch, U101 XC6206P332MR, U102 STM32F072CBTx, U301 74LVC1G125

Commit message: added pcb cutouts for mounting
Routing:
- net ROTA: track 250.0 -> 245.3 mm
- net ROTB: track 253.1 -> 248.3 mm
- net GND: track 846.4 -> 841.7 mm
- net ROW0: track 419.5 -> 422.5 mm
- net COL14: track 230.2 -> 228.9 mm
- net COL13: track 216.1 -> 214.9 mm
- net COL12: track 200.8 -> 199.7 mm
- net LED-: track 1815.8 -> 1814.8 mm
- net Net-(C113-Pad1): track 13.2 -> 13.7 mm
- net Net-(D302-Pad1): track 36.7 -> 36.2 mm
Other:
- board size 308.8 x 123.5 mm -> 308.3 x 123 mm
- net class Power: trace_width 0.3048 -> 0.508
- board text added: "isometric75 rev 1.0 github.com/ebastler/isometria-75 mpwr.xyz"
- board text removed: "isometric75 rev 1.0 github.com/ebastler/isometric-75 mpwr.xyz"
