File: isometria-75-pcb-iso/isometria-75-pcb-iso.kicad_pcb (KiCad board)
At the start: 2 copper layers, 308.3 x 123 mm, 320 parts, among them J101 USB, J102 SPI, J103 Conn_01x01_Male, Q101 AO3400A, SW101 RST, SW102 BOOT, SW201 Rotary_Encoder_Switch, U101 XC6206P332MR, U102 STM32F072CBTx, U301 74LVC1G125

Commit message: added manufacturing files
Parts:
- C101, C102: value 100u -> 100uF
- C103: value 10u -> 10uF
- C104, C106: value 1u -> 1uF
- C105, C111, C112: value 4.7u -> 4.7uF
- C107, C108, C109, C110, C113, C114, C115, C116, C117, C201, C202, C301, C302, C303, C304, C305, C306, C307, C308, C309, C310, C311, C312, C313, C314, C315, C316, C317, C318: value 100n -> 100nF
- R101: value 100 -> 100R
- R102: value 10 -> 10R
- R201, R202, R203, R204, R205, R206, R207, R208, R209, R210, R211, R212, R213, R214, R215, R216, R217, R218, R219, R220, R221, R222, R223, R224, R225, R226, R227, R228, R229, R230, R231, R232, R233, R234, R235, R236, R237, R238, R239, R240, R241, R242, R243, R244, R245, R246, R247, R248, R249, R250, R251, R252, R253, R254, R255, R256, R257, R258, R259, R260, R261, R262, R263, R264, R265, R266, R267, R268, R269, R270, R271, R272, R273, R274, R275, R276, R277, R278, R279, R280, R281, R282: value 680 -> 680R

Commit message: fixed minor bugs, migrated to new libs
Parts:
- removed R102: 10R, Resistor_SMD:R_0402_1005Metric
- added R2: 10k, Resistor_SMD:R_0402_1005Metric, B.Cu at (146.3, 101.6)
- SW1: renamed from SW101; footprint random-keyboard-parts:SKQG-1155865 -> Button_Switch_SMD:SW_SPST_SKQG_WithStem
- SW2: renamed from SW102; footprint random-keyboard-parts:SKQG-1155865 -> Button_Switch_SMD:SW_SPST_SKQG_WithStem
- turned SW1 to 90 degrees
- turned SW2 to 90 degrees
- renumbered C101 to C1, C110 to C10, C111 to C11, C112 to C12, C113 to C13, C114 to C14, C115 to C15, C116 to C16, C117 to C17, C201 to C18, C202 to C19, C102 to C2, C301 to C20, C302 to C21, C303 to C22, C304 to C23, C305 to C24, C306 to C25, C307 to C26, C308 to C27, C309 to C28, C310 to C29, C103 to C3, C311 to C30, C312 to C31, C313 to C32, C314 to C33, C315 to C34, C316 to C35, C317 to C36, C318 to C37, C104 to C4, C105 to C5, C106 to C6, C107 to C7, C108 to C8, C109 to C9, D201 to D1, D252 to D10, D317 to D100, D258 to D11, D264 to D12, D268 to D13, D273 to D14, D278 to D15, D202 to D16, D208 to D17, D212 to D18, D218 to D19, D207 to D2, D223 to D20, D227 to D21, D232 to D22, D238 to D23, D243 to D24, D248 to D25, D253 to D26, D259 to D27, D265 to D28, D274 to D29, D211 to D3, D279 to D30, D203 to D31, D213 to D32, D219 to D33, D224 to D34, D228 to D35, D233 to D36, D239 to D37, D244 to D38, D249 to D39, D217 to D4, D254 to D40, D260 to D41, D266 to D42, D269 to D43, D280 to D44, D204 to D45, D214 to D46, D220 to D47, D225 to D48, D229 to D49, D222 to D5, D234 to D50, D240 to D51, D245 to D52, D250 to D53, D255 to D54, D261 to D55, D267 to D56, D270 to D57, D275 to D58, D281 to D59, D231 to D6, D205 to D60, D209 to D61, D215 to D62, D221 to D63, D226 to D64, D230 to D65, D235 to D66, D241 to D67, D246 to D68, D251 to D69, D237 to D7, D256 to D70, D262 to D71, D271 to D72, D276 to D73, D282 to D74, D206 to D75, D210 to D76, D216 to D77, D236 to D78, D257 to D79, D242 to D8, D263 to D80, D272 to D81, D277 to D82, D283 to D83, D301 to D84, D302 to D85, D303 to D86, D304 to D87, D305 to D88, D306 to D89, D247 to D9, D307 to D90, D308 to D91, D309 to D92, D310 to D93, D311 to D94, D312 to D95, D313 to D96, D314 to D97, D315 to D98, D316 to D99, J101 to J1, J102 to J2, J103 to J3, MX201 to MX1, MX252 to MX10, MX258 to MX11, MX264 to MX12, MX268 to MX13, MX273 to MX14, MX202 to MX15, MX208 to MX16, MX212 to MX17, MX218 to MX18, MX223 to MX19, MX207 to MX2, MX227 to MX20, MX232 to MX21, MX238 to MX22, MX243 to MX23, MX248 to MX24, MX253 to MX25, MX259 to MX26, MX265 to MX27, MX274 to MX28, MX278 to MX29, MX211 to MX3, MX203 to MX30, MX213 to MX31, MX219 to MX32, MX224 to MX33, MX228 to MX34, MX233 to MX35, MX239 to MX36, MX244 to MX37, MX249 to MX38, MX254 to MX39, MX217 to MX4, MX260 to MX40, MX266 to MX41, MX269 to MX42, MX279 to MX43, MX204 to MX44, MX214 to MX45, MX220 to MX46, MX225 to MX47, MX229 to MX48, MX234 to MX49, MX222 to MX5, MX240 to MX50, MX245 to MX51, MX250 to MX52, MX255 to MX53, MX261 to MX54, MX267 to MX55, MX270 to MX56, MX275 to MX57, MX280 to MX58, MX205 to MX59, MX231 to MX6, MX209 to MX60, MX215 to MX61, MX221 to MX62, MX226 to MX63, MX230 to MX64, MX235 to MX65, MX241 to MX66, MX246 to MX67, MX251 to MX68, MX256 to MX69, MX237 to MX7, MX262 to MX70, MX271 to MX71, MX276 to MX72, MX281 to MX73, MX206 to MX74, MX210 to MX75, MX216 to MX76, MX236 to MX77, MX257 to MX78, MX263 to MX79, MX242 to MX8, MX272 to MX80, MX277 to MX81, MX282 to MX82, MX247 to MX9, Q101 to Q1, R101 to R1, R207 to R10, R211 to R11, R217 to R12, R222 to R13, R231 to R14, R237 to R15, R242 to R16, R247 to R17, R252 to R18, R258 to R19, R264 to R20, R268 to R21, R273 to R22, R284 to R23, R202 to R24, R208 to R25, R212 to R26, R218 to R27, R223 to R28, R227 to R29, R103 to R3, R232 to R30, R238 to R31, R243 to R32, R248 to R33, R253 to R34, R259 to R35, R265 to R36, R274 to R37, R278 to R38, R203 to R39, R104 to R4, R213 to R40, R219 to R41, R224 to R42, R228 to R43, R233 to R44, R239 to R45, R244 to R46, R249 to R47, R254 to R48, R260 to R49, R105 to R5, R266 to R50, R269 to R51, R279 to R52, R204 to R53, R214 to R54, R220 to R55, R225 to R56, R229 to R57, R234 to R58, R240 to R59, R106 to R6, R245 to R60, R250 to R61, R255 to R62, R261 to R63, R267 to R64, R270 to R65, R275 to R66, R280 to R67, R205 to R68, R209 to R69, R107 to R7, R215 to R70, R221 to R71, R226 to R72, R230 to R73, R235 to R74, R241 to R75, R246 to R76, R251 to R77, R256 to R78, R262 to R79, R283 to R8, R271 to R80, R276 to R81, R281 to R82, R206 to R83, R210 to R84, R216 to R85, R236 to R86, R257 to R87, R263 to R88, R272 to R89, R201 to R9, R277 to R90, R282 to R91, SW201 to SW3, U101 to U1, U102 to U2, U301 to U3
Connections:
- C14 pad 1: /VDDA -> +3V3
- U2 pad 9: /VDDA -> +3V3
Routing:
- net +3V3: track 160.1 -> 172.2 mm
- net /BOOT: track 81.0 -> 88.4 mm
- net /RST: track 103.4 -> 109.8 mm
- net /VDDA: track 6.06 -> 0.00 mm
- net LED_PWM: track 8.00 -> 9.10 mm

Commit message: added branding submodule
Parts:
- added G***: LOGO, logo-branding:logo_silk_15, B.Cu at (276.2, 74.8)

Commit message: added logo to pcb
Parts:
- removed the G*** at (276.2, 74.8)
- added G***: LOGO, logo-branding:logo_silk_7p5, B.Cu at (278.8, 71.8)

Commit message: updated rev numbering
Other:
- board text added: "isometria75 rev 1.1 github.com/ebastler/isometria-75 mpwr.xyz"
- board text removed: "isometria75 rev 1.0 github.com/ebastler/isometria-75 mpwr.xyz"
