File: isometria-75-pcb-iso/isometria-75-pcb-ml.sch (KiCad schematic (older format))
At the start: 15 parts, among them J1 USB, Q1 AO3400A, U1 TXB0101, U2 XC6206P332MR, U3 nRF52840_holyiot_18010

Commit message: began renaming project
Parts:
- added J2: SWD, Connector_PinHeader_2.54mm:PinHeader_1x03_P2.54mm_Vertical, symbol Connector:Conn_01x03_Male
- added Q2: AO3401A, Package_TO_SOT_SMD:SOT-23, symbol Transistor_FET:AO3401A
- added Q3: 2N7002, Package_TO_SOT_SMD:SOT-23, symbol Transistor_FET:2N7002
- added R4, R6: 10k, Resistor_SMD:R_0603_1608Metric_Pad1.05x0.95mm_HandSolder, symbol Device:R_Small
- added R5: 100R, Resistor_SMD:R_0603_1608Metric_Pad1.05x0.95mm_HandSolder, symbol Device:R_Small
- added R7: 1.3M, Resistor_SMD:R_0603_1608Metric_Pad1.05x0.95mm_HandSolder, symbol Device:R_Small
- added R8: 2M, Resistor_SMD:R_0603_1608Metric_Pad1.05x0.95mm_HandSolder, symbol Device:R_Small
Connections:
- net labels added: SWDCLK, UG_EN, UG_PWR, VSENSE
- net labels removed: SPI_CS, SPI_IRQ, SPI_MISO, SPI_MOSI, SPI_RES, SPI_SCK
- wire segments 49 -> 71
Other:
- note added: "Cut underglow power for battery life"
- note added: "Isometria⁷⁵ - 75% multilayout wireless keyboard"
- note removed: "Isometria⁷⁵ - 75% blocked ISO layout keyboard"
- moved on the sheet: C3, C4, C5, C6, C7, U2
