File: isometria-75-pcb-iso/matrix.sch (KiCad schematic (older format))
At the start: 252 parts, among them SW201 Rotary_Encoder_Switch

Commit message: fixed minor bugs, migrated to new libs
Parts:
- renumbered C201 to C18, C202 to C19, D201 to D1, D252 to D10, D258 to D11, D264 to D12, D268 to D13, D273 to D14, D278 to D15, D202 to D16, D208 to D17, D212 to D18, D218 to D19, D207 to D2, D223 to D20, D227 to D21, D232 to D22, D238 to D23, D243 to D24, D248 to D25, D253 to D26, D259 to D27, D265 to D28, D274 to D29, D211 to D3, D279 to D30, D203 to D31, D213 to D32, D219 to D33, D224 to D34, D228 to D35, D233 to D36, D239 to D37, D244 to D38, D249 to D39, D217 to D4, D254 to D40, D260 to D41, D266 to D42, D269 to D43, D280 to D44, D204 to D45, D214 to D46, D220 to D47, D225 to D48, D229 to D49, D222 to D5, D234 to D50, D240 to D51, D245 to D52, D250 to D53, D255 to D54, D261 to D55, D267 to D56, D270 to D57, D275 to D58, D281 to D59, D231 to D6, D205 to D60, D209 to D61, D215 to D62, D221 to D63, D226 to D64, D230 to D65, D235 to D66, D241 to D67, D246 to D68, D251 to D69, D237 to D7, D256 to D70, D262 to D71, D271 to D72, D276 to D73, D282 to D74, D206 to D75, D210 to D76, D216 to D77, D236 to D78, D257 to D79, D242 to D8, D263 to D80, D272 to D81, D277 to D82, D283 to D83, D247 to D9, MX201 to MX1, MX252 to MX10, MX258 to MX11, MX264 to MX12, MX268 to MX13, MX273 to MX14, MX202 to MX15, MX208 to MX16, MX212 to MX17, MX218 to MX18, MX223 to MX19, MX207 to MX2, MX227 to MX20, MX232 to MX21, MX238 to MX22, MX243 to MX23, MX248 to MX24, MX253 to MX25, MX259 to MX26, MX265 to MX27, MX274 to MX28, MX278 to MX29, MX211 to MX3, MX203 to MX30, MX213 to MX31, MX219 to MX32, MX224 to MX33, MX228 to MX34, MX233 to MX35, MX239 to MX36, MX244 to MX37, MX249 to MX38, MX254 to MX39, MX217 to MX4, MX260 to MX40, MX266 to MX41, MX269 to MX42, MX279 to MX43, MX204 to MX44, MX214 to MX45, MX220 to MX46, MX225 to MX47, MX229 to MX48, MX234 to MX49, MX222 to MX5, MX240 to MX50, MX245 to MX51, MX250 to MX52, MX255 to MX53, MX261 to MX54, MX267 to MX55, MX270 to MX56, MX275 to MX57, MX280 to MX58, MX205 to MX59, MX231 to MX6, MX209 to MX60, MX215 to MX61, MX221 to MX62, MX226 to MX63, MX230 to MX64, MX235 to MX65, MX241 to MX66, MX246 to MX67, MX251 to MX68, MX256 to MX69, MX237 to MX7, MX262 to MX70, MX271 to MX71, MX276 to MX72, MX281 to MX73, MX206 to MX74, MX210 to MX75, MX216 to MX76, MX236 to MX77, MX257 to MX78, MX263 to MX79, MX242 to MX8, MX272 to MX80, MX277 to MX81, MX282 to MX82, MX247 to MX9, R207 to R10, R211 to R11, R217 to R12, R222 to R13, R231 to R14, R237 to R15, R242 to R16, R247 to R17, R252 to R18, R258 to R19, R264 to R20, R268 to R21, R273 to R22, R284 to R23, R202 to R24, R208 to R25, R212 to R26, R218 to R27, R223 to R28, R227 to R29, R232 to R30, R238 to R31, R243 to R32, R248 to R33, R253 to R34, R259 to R35, R265 to R36, R274 to R37, R278 to R38, R203 to R39, R213 to R40, R219 to R41, R224 to R42, R228 to R43, R233 to R44, R239 to R45, R244 to R46, R249 to R47, R254 to R48, R260 to R49, R266 to R50, R269 to R51, R279 to R52, R204 to R53, R214 to R54, R220 to R55, R225 to R56, R229 to R57, R234 to R58, R240 to R59, R245 to R60, R250 to R61, R255 to R62, R261 to R63, R267 to R64, R270 to R65, R275 to R66, R280 to R67, R205 to R68, R209 to R69, R215 to R70, R221 to R71, R226 to R72, R230 to R73, R235 to R74, R241 to R75, R246 to R76, R251 to R77, R256 to R78, R262 to R79, R283 to R8, R271 to R80, R276 to R81, R281 to R82, R206 to R83, R210 to R84, R216 to R85, R236 to R86, R257 to R87, R263 to R88, R272 to R89, R201 to R9, R277 to R90, R282 to R91, SW201 to SW3

Commit message: started nRF v2 rework
Parts:
- removed D1, D10, D11, D12, D13, D14, D15, D16, D17, D18, D19, D2, D20, D21, D22, D23, D24, D25, D26, D27, D28, D29, D3, D30, D31, D32, D33, D34, D35, D36, D37, D38, D39, D4, D40, D41, D42, D43, D44, D45, D46, D47, D48, D49, D5, D50, D51, D52, D53, D54, D55, D56, D57, D58, D59, D6, D60, D61, D62, D63, D64, D65, D66, D67, D68, D69, D7, D70, D71, D72, D73, D74, D75, D76, D77, D78, D79, D8, D80, D81, D82, D83, D9: 1N4148, Diode_SMD:D_SOD-323F, symbol Device:D_Small
- added D1, D10, D11, D12, D13, D14, D15, D16, D17, D18, D19, D2, D20, D21, D22, D23, D24, D25, D26, D27, D28, D29, D3, D30, D31, D32, D33, D34, D35, D36, D37, D38, D39, D4, D40, D41, D42, D43, D44, D45, D5, D6, D7, D8, D9: BAV70, Package_TO_SOT_SMD:SOT-23, symbol Diode:BAV70
- added MX43: /_ansi, MX_Only:MXOnly-1.5U, symbol MX_Alps_Hybrid:MX-LED
- added MX59: enter_ansi, MX_Only:MXOnly-2.25U, symbol MX_Alps_Hybrid:MX-LED
- added MX62: shift_ansi, MX_Only:MXOnly-2.25U, symbol MX_Alps_Hybrid:MX-LED
- C8: renamed from C18; footprint Capacitor_SMD:C_0402_1005Metric -> Capacitor_SMD:C_0603_1608Metric_Pad1.05x0.95mm_HandSolder
- C9: renamed from C19; footprint Capacitor_SMD:C_0402_1005Metric -> Capacitor_SMD:C_0603_1608Metric_Pad1.05x0.95mm_HandSolder
- MX57: renamed from MX56; value MX-LED -> nuhs
- MX58: renamed from MX57; value MX-LED -> enter_iso; footprint MX_Only:MXOnly-ISO -> MX_Only:MXOnly-ISO-ROTATED
- MX61: renamed from MX59; value MX-LED -> shift_iso
- MX63: renamed from MX60; value MX-LED -> nubs
- R10: renamed from R14; footprint Resistor_SMD:R_0603_1608Metric -> Resistor_SMD:R_0603_1608Metric_Pad1.05x0.95mm_HandSolder
- R11: renamed from R15; footprint Resistor_SMD:R_0603_1608Metric -> Resistor_SMD:R_0603_1608Metric_Pad1.05x0.95mm_HandSolder
- R12: renamed from R16; footprint Resistor_SMD:R_0603_1608Metric -> Resistor_SMD:R_0603_1608Metric_Pad1.05x0.95mm_HandSolder
- R13: renamed from R17; footprint Resistor_SMD:R_0603_1608Metric -> Resistor_SMD:R_0603_1608Metric_Pad1.05x0.95mm_HandSolder
- R14: renamed from R18; footprint Resistor_SMD:R_0603_1608Metric -> Resistor_SMD:R_0603_1608Metric_Pad1.05x0.95mm_HandSolder
- R15: renamed from R19; footprint Resistor_SMD:R_0603_1608Metric -> Resistor_SMD:R_0603_1608Metric_Pad1.05x0.95mm_HandSolder
- R16: renamed from R20; footprint Resistor_SMD:R_0603_1608Metric -> Resistor_SMD:R_0603_1608Metric_Pad1.05x0.95mm_HandSolder
- R17: renamed from R21; footprint Resistor_SMD:R_0603_1608Metric -> Resistor_SMD:R_0603_1608Metric_Pad1.05x0.95mm_HandSolder
- R18: renamed from R22; footprint Resistor_SMD:R_0603_1608Metric -> Resistor_SMD:R_0603_1608Metric_Pad1.05x0.95mm_HandSolder
- R19: renamed from R23; footprint Resistor_SMD:R_0402_1005Metric -> Resistor_SMD:R_0603_1608Metric_Pad1.05x0.95mm_HandSolder
- R20: renamed from R24; footprint Resistor_SMD:R_0603_1608Metric -> Resistor_SMD:R_0603_1608Metric_Pad1.05x0.95mm_HandSolder
- R21: renamed from R25; footprint Resistor_SMD:R_0603_1608Metric -> Resistor_SMD:R_0603_1608Metric_Pad1.05x0.95mm_HandSolder
- R22: renamed from R26; footprint Resistor_SMD:R_0603_1608Metric -> Resistor_SMD:R_0603_1608Metric_Pad1.05x0.95mm_HandSolder
- R23: renamed from R27; footprint Resistor_SMD:R_0603_1608Metric -> Resistor_SMD:R_0603_1608Metric_Pad1.05x0.95mm_HandSolder
- R24: renamed from R28; footprint Resistor_SMD:R_0603_1608Metric -> Resistor_SMD:R_0603_1608Metric_Pad1.05x0.95mm_HandSolder
- R25: renamed from R29; footprint Resistor_SMD:R_0603_1608Metric -> Resistor_SMD:R_0603_1608Metric_Pad1.05x0.95mm_HandSolder
- R26: renamed from R30; footprint Resistor_SMD:R_0603_1608Metric -> Resistor_SMD:R_0603_1608Metric_Pad1.05x0.95mm_HandSolder
- R27: renamed from R31; footprint Resistor_SMD:R_0603_1608Metric -> Resistor_SMD:R_0603_1608Metric_Pad1.05x0.95mm_HandSolder
- R28: renamed from R32; footprint Resistor_SMD:R_0603_1608Metric -> Resistor_SMD:R_0603_1608Metric_Pad1.05x0.95mm_HandSolder
- R29: renamed from R33; footprint Resistor_SMD:R_0603_1608Metric -> Resistor_SMD:R_0603_1608Metric_Pad1.05x0.95mm_HandSolder
- R30: renamed from R34; footprint Resistor_SMD:R_0603_1608Metric -> Resistor_SMD:R_0603_1608Metric_Pad1.05x0.95mm_HandSolder
- R31: renamed from R35; footprint Resistor_SMD:R_0603_1608Metric -> Resistor_SMD:R_0603_1608Metric_Pad1.05x0.95mm_HandSolder
- R32: renamed from R36; footprint Resistor_SMD:R_0603_1608Metric -> Resistor_SMD:R_0603_1608Metric_Pad1.05x0.95mm_HandSolder
- R33: renamed from R37; footprint Resistor_SMD:R_0603_1608Metric -> Resistor_SMD:R_0603_1608Metric_Pad1.05x0.95mm_HandSolder
- R34: renamed from R38; footprint Resistor_SMD:R_0603_1608Metric -> Resistor_SMD:R_0603_1608Metric_Pad1.05x0.95mm_HandSolder
- R35: renamed from R39; footprint Resistor_SMD:R_0603_1608Metric -> Resistor_SMD:R_0603_1608Metric_Pad1.05x0.95mm_HandSolder
- R36: renamed from R40; footprint Resistor_SMD:R_0603_1608Metric -> Resistor_SMD:R_0603_1608Metric_Pad1.05x0.95mm_HandSolder
- R37: renamed from R41; footprint Resistor_SMD:R_0603_1608Metric -> Resistor_SMD:R_0603_1608Metric_Pad1.05x0.95mm_HandSolder
- R38: renamed from R42; footprint Resistor_SMD:R_0603_1608Metric -> Resistor_SMD:R_0603_1608Metric_Pad1.05x0.95mm_HandSolder
- R39: renamed from R43; footprint Resistor_SMD:R_0603_1608Metric -> Resistor_SMD:R_0603_1608Metric_Pad1.05x0.95mm_HandSolder
- R4: renamed from R8; footprint Resistor_SMD:R_0402_1005Metric -> Resistor_SMD:R_0603_1608Metric_Pad1.05x0.95mm_HandSolder
- R40: renamed from R44; footprint Resistor_SMD:R_0603_1608Metric -> Resistor_SMD:R_0603_1608Metric_Pad1.05x0.95mm_HandSolder
- R41: renamed from R45; footprint Resistor_SMD:R_0603_1608Metric -> Resistor_SMD:R_0603_1608Metric_Pad1.05x0.95mm_HandSolder
- R42: renamed from R46; footprint Resistor_SMD:R_0603_1608Metric -> Resistor_SMD:R_0603_1608Metric_Pad1.05x0.95mm_HandSolder
- R43: renamed from R47; footprint Resistor_SMD:R_0603_1608Metric -> Resistor_SMD:R_0603_1608Metric_Pad1.05x0.95mm_HandSolder
- R44: renamed from R48; footprint Resistor_SMD:R_0603_1608Metric -> Resistor_SMD:R_0603_1608Metric_Pad1.05x0.95mm_HandSolder
- R45: renamed from R49; footprint Resistor_SMD:R_0603_1608Metric -> Resistor_SMD:R_0603_1608Metric_Pad1.05x0.95mm_HandSolder
- R46: renamed from R50; footprint Resistor_SMD:R_0603_1608Metric -> Resistor_SMD:R_0603_1608Metric_Pad1.05x0.95mm_HandSolder
- R47: renamed from R51; footprint Resistor_SMD:R_0603_1608Metric -> Resistor_SMD:R_0603_1608Metric_Pad1.05x0.95mm_HandSolder
- R48: renamed from R52; footprint Resistor_SMD:R_0603_1608Metric -> Resistor_SMD:R_0603_1608Metric_Pad1.05x0.95mm_HandSolder
- R49: renamed from R53; footprint Resistor_SMD:R_0603_1608Metric -> Resistor_SMD:R_0603_1608Metric_Pad1.05x0.95mm_HandSolder
- R5: renamed from R9; footprint Resistor_SMD:R_0603_1608Metric -> Resistor_SMD:R_0603_1608Metric_Pad1.05x0.95mm_HandSolder
- R50: renamed from R54; footprint Resistor_SMD:R_0603_1608Metric -> Resistor_SMD:R_0603_1608Metric_Pad1.05x0.95mm_HandSolder
- R51: renamed from R55; footprint Resistor_SMD:R_0603_1608Metric -> Resistor_SMD:R_0603_1608Metric_Pad1.05x0.95mm_HandSolder
- R52: renamed from R56; footprint Resistor_SMD:R_0603_1608Metric -> Resistor_SMD:R_0603_1608Metric_Pad1.05x0.95mm_HandSolder
- R53: renamed from R57; footprint Resistor_SMD:R_0603_1608Metric -> Resistor_SMD:R_0603_1608Metric_Pad1.05x0.95mm_HandSolder
- R54: renamed from R58; footprint Resistor_SMD:R_0603_1608Metric -> Resistor_SMD:R_0603_1608Metric_Pad1.05x0.95mm_HandSolder
- R55: renamed from R59; footprint Resistor_SMD:R_0603_1608Metric -> Resistor_SMD:R_0603_1608Metric_Pad1.05x0.95mm_HandSolder
- R56: renamed from R60; footprint Resistor_SMD:R_0603_1608Metric -> Resistor_SMD:R_0603_1608Metric_Pad1.05x0.95mm_HandSolder
- R57: renamed from R61; footprint Resistor_SMD:R_0603_1608Metric -> Resistor_SMD:R_0603_1608Metric_Pad1.05x0.95mm_HandSolder
- R58: renamed from R62; footprint Resistor_SMD:R_0603_1608Metric -> Resistor_SMD:R_0603_1608Metric_Pad1.05x0.95mm_HandSolder
- R59: renamed from R63; footprint Resistor_SMD:R_0603_1608Metric -> Resistor_SMD:R_0603_1608Metric_Pad1.05x0.95mm_HandSolder
- R6: renamed from R10; footprint Resistor_SMD:R_0603_1608Metric -> Resistor_SMD:R_0603_1608Metric_Pad1.05x0.95mm_HandSolder
- R60: renamed from R64; footprint Resistor_SMD:R_0603_1608Metric -> Resistor_SMD:R_0603_1608Metric_Pad1.05x0.95mm_HandSolder
- R61: renamed from R65; footprint Resistor_SMD:R_0603_1608Metric -> Resistor_SMD:R_0603_1608Metric_Pad1.05x0.95mm_HandSolder
- R62: renamed from R66; footprint Resistor_SMD:R_0603_1608Metric -> Resistor_SMD:R_0603_1608Metric_Pad1.05x0.95mm_HandSolder
- R63: renamed from R67; footprint Resistor_SMD:R_0603_1608Metric -> Resistor_SMD:R_0603_1608Metric_Pad1.05x0.95mm_HandSolder
- R64: renamed from R68; footprint Resistor_SMD:R_0603_1608Metric -> Resistor_SMD:R_0603_1608Metric_Pad1.05x0.95mm_HandSolder
- R65: renamed from R69; footprint Resistor_SMD:R_0603_1608Metric -> Resistor_SMD:R_0603_1608Metric_Pad1.05x0.95mm_HandSolder
- R66: renamed from R70; footprint Resistor_SMD:R_0603_1608Metric -> Resistor_SMD:R_0603_1608Metric_Pad1.05x0.95mm_HandSolder
- R67: renamed from R71; footprint Resistor_SMD:R_0603_1608Metric -> Resistor_SMD:R_0603_1608Metric_Pad1.05x0.95mm_HandSolder
- R68: renamed from R72; footprint Resistor_SMD:R_0603_1608Metric -> Resistor_SMD:R_0603_1608Metric_Pad1.05x0.95mm_HandSolder
- R69: renamed from R73; footprint Resistor_SMD:R_0603_1608Metric -> Resistor_SMD:R_0603_1608Metric_Pad1.05x0.95mm_HandSolder
- R7: renamed from R11; footprint Resistor_SMD:R_0603_1608Metric -> Resistor_SMD:R_0603_1608Metric_Pad1.05x0.95mm_HandSolder
- R70: renamed from R74; footprint Resistor_SMD:R_0603_1608Metric -> Resistor_SMD:R_0603_1608Metric_Pad1.05x0.95mm_HandSolder
- R71: renamed from R75; footprint Resistor_SMD:R_0603_1608Metric -> Resistor_SMD:R_0603_1608Metric_Pad1.05x0.95mm_HandSolder
- R72: renamed from R76; footprint Resistor_SMD:R_0603_1608Metric -> Resistor_SMD:R_0603_1608Metric_Pad1.05x0.95mm_HandSolder
- R73: renamed from R77; footprint Resistor_SMD:R_0603_1608Metric -> Resistor_SMD:R_0603_1608Metric_Pad1.05x0.95mm_HandSolder
- R74: renamed from R78; footprint Resistor_SMD:R_0603_1608Metric -> Resistor_SMD:R_0603_1608Metric_Pad1.05x0.95mm_HandSolder
- R75: renamed from R79; footprint Resistor_SMD:R_0603_1608Metric -> Resistor_SMD:R_0603_1608Metric_Pad1.05x0.95mm_HandSolder
- R76: renamed from R80; footprint Resistor_SMD:R_0603_1608Metric -> Resistor_SMD:R_0603_1608Metric_Pad1.05x0.95mm_HandSolder
- R77: renamed from R81; footprint Resistor_SMD:R_0603_1608Metric -> Resistor_SMD:R_0603_1608Metric_Pad1.05x0.95mm_HandSolder
- R78: renamed from R82; footprint Resistor_SMD:R_0603_1608Metric -> Resistor_SMD:R_0603_1608Metric_Pad1.05x0.95mm_HandSolder
- R79: renamed from R83; footprint Resistor_SMD:R_0603_1608Metric -> Resistor_SMD:R_0603_1608Metric_Pad1.05x0.95mm_HandSolder
- R8: renamed from R12; footprint Resistor_SMD:R_0603_1608Metric -> Resistor_SMD:R_0603_1608Metric_Pad1.05x0.95mm_HandSolder
- R80: renamed from R84; footprint Resistor_SMD:R_0603_1608Metric -> Resistor_SMD:R_0603_1608Metric_Pad1.05x0.95mm_HandSolder
- R81: renamed from R85; footprint Resistor_SMD:R_0603_1608Metric -> Resistor_SMD:R_0603_1608Metric_Pad1.05x0.95mm_HandSolder
- R82: renamed from R86; footprint Resistor_SMD:R_0603_1608Metric -> Resistor_SMD:R_0603_1608Metric_Pad1.05x0.95mm_HandSolder
- R83: renamed from R87; footprint Resistor_SMD:R_0603_1608Metric -> Resistor_SMD:R_0603_1608Metric_Pad1.05x0.95mm_HandSolder
- R84: renamed from R88; footprint Resistor_SMD:R_0603_1608Metric -> Resistor_SMD:R_0603_1608Metric_Pad1.05x0.95mm_HandSolder
- R85: renamed from R89; footprint Resistor_SMD:R_0603_1608Metric -> Resistor_SMD:R_0603_1608Metric_Pad1.05x0.95mm_HandSolder
- R86: renamed from R90; footprint Resistor_SMD:R_0603_1608Metric -> Resistor_SMD:R_0603_1608Metric_Pad1.05x0.95mm_HandSolder
- R87: renamed from R91; footprint Resistor_SMD:R_0603_1608Metric -> Resistor_SMD:R_0603_1608Metric_Pad1.05x0.95mm_HandSolder
- R9: renamed from R13; footprint Resistor_SMD:R_0603_1608Metric -> Resistor_SMD:R_0603_1608Metric_Pad1.05x0.95mm_HandSolder
- renumbered MX43 to MX44, MX44 to MX45, MX45 to MX46, MX46 to MX47, MX47 to MX48, MX48 to MX49, MX49 to MX50, MX50 to MX51, MX51 to MX52, MX52 to MX53, MX53 to MX54, MX54 to MX55, MX55 to MX56, MX58 to MX60, MX61 to MX64, MX62 to MX65, MX63 to MX66, MX64 to MX67, MX65 to MX68, MX66 to MX69, MX67 to MX70, MX68 to MX71, MX69 to MX72, MX70 to MX73, MX71 to MX74, MX72 to MX75, MX73 to MX76, MX74 to MX77, MX75 to MX78, MX76 to MX79, MX77 to MX80, MX78 to MX81, MX79 to MX82, MX80 to MX83, MX81 to MX84, MX82 to MX85, SW3 to SW1
Connections:
- net +5V: no longer MX1.4 (LEDGND), MX10.4 (LEDGND), MX11.4 (LEDGND), MX12.4 (LEDGND), MX13.4 (LEDGND), MX14.4 (LEDGND), MX15.4 (LEDGND), MX16.4 (LEDGND), MX17.4 (LEDGND), MX18.4 (LEDGND), MX19.4 (LEDGND), MX2.4 (LEDGND), MX20.4 (LEDGND), MX21.4 (LEDGND), MX22.4 (LEDGND), MX23.4 (LEDGND), MX24.4 (LEDGND), MX25.4 (LEDGND), MX26.4 (LEDGND), MX27.4 (LEDGND), MX28.4 (LEDGND), MX29.4 (LEDGND), MX3.4 (LEDGND), MX30.4 (LEDGND), MX31.4 (LEDGND), MX32.4 (LEDGND), MX33.4 (LEDGND), MX34.4 (LEDGND), MX35.4 (LEDGND), MX36.4 (LEDGND), MX37.4 (LEDGND), MX38.4 (LEDGND), MX39.4 (LEDGND), MX4.4 (LEDGND), MX40.4 (LEDGND), MX41.4 (LEDGND), MX42.4 (LEDGND), MX44.4 (LEDGND), MX45.4 (LEDGND), MX46.4 (LEDGND), MX47.4 (LEDGND), MX48.4 (LEDGND), MX49.4 (LEDGND), MX5.4 (LEDGND), MX50.4 (LEDGND), MX51.4 (LEDGND), MX52.4 (LEDGND), MX53.4 (LEDGND), MX54.4 (LEDGND), MX55.4 (LEDGND), MX56.4 (LEDGND), MX57.4 (LEDGND), MX58.4 (LEDGND), MX6.4 (LEDGND), MX60.4 (LEDGND), MX61.4 (LEDGND), MX63.4 (LEDGND), MX64.4 (LEDGND), MX65.4 (LEDGND), MX66.4 (LEDGND), MX67.4 (LEDGND), MX68.4 (LEDGND), MX69.4 (LEDGND), MX7.4 (LEDGND), MX70.4 (LEDGND), MX71.4 (LEDGND), MX72.4 (LEDGND), MX73.4 (LEDGND), MX74.4 (LEDGND), MX75.4 (LEDGND), MX76.4 (LEDGND), MX77.4 (LEDGND), MX78.4 (LEDGND), MX79.4 (LEDGND), MX8.4 (LEDGND), MX80.4 (LEDGND), MX81.4 (LEDGND), MX82.4 (LEDGND), MX83.4 (LEDGND), MX84.4 (LEDGND), MX85.4 (LEDGND), MX9.4 (LEDGND)
- net COL0: no longer MX1.1 (COL), MX15.1 (COL), MX30.1 (COL), MX45.1 (COL), MX61.1 (COL), MX77.1 (COL)
- net COL1: no longer MX16.1 (COL), MX2.1 (COL), MX63.1 (COL), MX78.1 (COL)
- net COL10: no longer MX10.1 (COL), MX25.1 (COL), MX39.1 (COL), MX54.1 (COL), MX72.1 (COL), MX81.1 (COL)
- net COL11: no longer MX11.1 (COL), MX26.1 (COL), MX40.1 (COL), MX55.1 (COL), MX73.1 (COL), MX82.1 (COL)
- net COL12: no longer MX12.1 (COL), MX27.1 (COL), MX41.1 (COL), MX56.1 (COL)
- net COL13: no longer MX13.1 (COL), MX42.1 (COL), MX57.1 (COL), MX74.1 (COL), MX83.1 (COL)
- net COL14: no longer MX14.1 (COL), MX28.1 (COL), MX58.1 (COL), MX75.1 (COL), MX84.1 (COL)
- net COL15: no longer MX29.1 (COL), MX44.1 (COL), MX60.1 (COL), MX76.1 (COL), MX85.1 (COL)
- net COL2: no longer MX17.1 (COL), MX3.1 (COL), MX31.1 (COL), MX46.1 (COL), MX64.1 (COL), MX79.1 (COL)
- net COL3: no longer MX18.1 (COL), MX32.1 (COL), MX4.1 (COL), MX47.1 (COL), MX65.1 (COL)
- net COL4: no longer MX19.1 (COL), MX33.1 (COL), MX48.1 (COL), MX5.1 (COL), MX66.1 (COL)
- net COL5: no longer MX20.1 (COL), MX34.1 (COL), MX49.1 (COL), MX67.1 (COL)
- net COL6: no longer MX21.1 (COL), MX35.1 (COL), MX50.1 (COL), MX6.1 (COL), MX68.1 (COL), MX80.1 (COL)
- net COL7: no longer MX22.1 (COL), MX36.1 (COL), MX51.1 (COL), MX69.1 (COL), MX7.1 (COL)
- net COL8: no longer MX23.1 (COL), MX37.1 (COL), MX52.1 (COL), MX70.1 (COL), MX8.1 (COL)
- net COL9: no longer MX24.1 (COL), MX38.1 (COL), MX53.1 (COL), MX71.1 (COL), MX9.1 (COL)
- net LED-: no longer R10.2, R11.2, R12.2, R13.2, R14.2, R15.2, R16.2, R17.2, R18.2, R20.2, R21.2, R22.2, R23.2, R24.2, R25.2, R26.2, R27.2, R28.2, R29.2, R30.2, R31.2, R32.2, R33.2, R34.2, R35.2, R36.2, R37.2, R38.2, R39.2, R40.2, R41.2, R42.2, R43.2, R44.2, R45.2, R46.2, R47.2, R48.2, R49.2, R5.2, R50.2, R51.2, R52.2, R53.2, R54.2, R55.2, R56.2, R57.2, R58.2, R59.2, R6.2, R60.2, R61.2, R62.2, R63.2, R64.2, R65.2, R66.2, R67.2, R68.2, R69.2, R7.2, R70.2, R71.2, R72.2, R73.2, R74.2, R75.2, R76.2, R77.2, R78.2, R79.2, R8.2, R80.2, R81.2, R82.2, R83.2, R84.2, R85.2, R86.2, R87.2, R9.2
- net at MX1.2 (ROW): now also D1.2 (A)
- net at MX15.2 (ROW): now also D9.2 (A)
- net at MX30.2 (ROW): now also D17.2 (A)
- net at MX45.2 (ROW): now also D25.2 (A)
- net at MX61.2 (ROW): now also D33.2 (A), MX62.2 (ROW)
- net at MX61.3 (LED), R64.1: now also MX62.3 (LED)
- net at MX77.2 (ROW): now also D41.2 (A)
- net at MX2.2 (ROW): now also D1.1 (A)
- net at MX16.2 (ROW): now also D9.1 (A)
- net at MX63.2 (ROW): now also D33.1 (A)
- net at MX78.2 (ROW): now also D41.1 (A)
- net at MX3.2 (ROW): now also D2.2 (A)
- net at MX17.2 (ROW): now also D10.2 (A)
- net at MX31.2 (ROW): now also D17.1 (A)
- net at MX46.2 (ROW): now also D25.1 (A)
- net at MX64.2 (ROW): now also D34.2 (A)
- net at MX79.2 (ROW): now also D42.2 (A)
- net at MX4.2 (ROW): now also D2.1 (A)
- net at MX18.2 (ROW): now also D10.1 (A)
- net at MX32.2 (ROW): now also D18.2 (A)
- net at MX47.2 (ROW): now also D26.2 (A)
- net at MX65.2 (ROW): now also D34.1 (A)
- net at MX5.2 (ROW): now also D3.1 (A)
- net at MX19.2 (ROW): now also D11.2 (A)
- net at MX33.2 (ROW): now also D18.1 (A)
- net at MX48.2 (ROW): now also D26.1 (A)
- net at MX66.2 (ROW): now also D35.2 (A)
- net at MX20.2 (ROW): now also D11.1 (A)
- net at MX34.2 (ROW): now also D19.2 (A)
- net at MX49.2 (ROW): now also D27.2 (A)
- net at MX67.2 (ROW): now also D35.1 (A)
- net at MX6.2 (ROW): now also D4.2 (A)
- net at MX21.2 (ROW): now also D12.2 (A)
- net at MX35.2 (ROW): now also D19.1 (A)
- net at MX50.2 (ROW): now also D27.1 (A)
- net at MX68.2 (ROW): now also D36.2 (A)
- net at MX80.2 (ROW): now also D42.1 (A)
- net at MX7.2 (ROW): now also D4.1 (A)
- net at MX22.2 (ROW): now also D12.1 (A)
- net at MX36.2 (ROW): now also D20.2 (A)
- net at MX51.2 (ROW): now also D28.2 (A)
- net at MX69.2 (ROW): now also D36.1 (A)
- net at MX8.2 (ROW): now also D5.2 (A)
- net at MX23.2 (ROW): now also D13.2 (A)
- net at MX37.2 (ROW): now also D20.1 (A)
- net at MX52.2 (ROW): now also D28.1 (A)
- net at MX70.2 (ROW): now also D37.2 (A)
- net at MX9.2 (ROW): now also D5.1 (A)
- net at MX24.2 (ROW): now also D13.1 (A)
- net at MX38.2 (ROW): now also D21.2 (A)
- net at MX53.2 (ROW): now also D29.2 (A)
- net at MX71.2 (ROW): now also D37.1 (A)
- net at MX10.2 (ROW): now also D6.2 (A)
- net at MX25.2 (ROW): now also D14.2 (A)
- net at MX39.2 (ROW): now also D21.1 (A)
- net at MX54.2 (ROW): now also D29.1 (A)
- net at MX72.2 (ROW): now also D38.2 (A)
- net at MX81.2 (ROW): now also D43.2 (A)
- net at MX11.2 (ROW): now also D6.1 (A)
- net at MX26.2 (ROW): now also D14.1 (A)
- net at MX40.2 (ROW): now also D22.2 (A)
- net at MX55.2 (ROW): now also D30.2 (A)
- net at MX73.2 (ROW): now also D38.1 (A)
- net at MX82.2 (ROW): now also D43.1 (A)
- net at MX12.2 (ROW): now also D7.2 (A)
- net at MX27.2 (ROW): now also D15.2 (A)
- net at MX41.2 (ROW): now also D22.1 (A)
- net at MX56.2 (ROW): now also D30.1 (A)
- net at MX13.2 (ROW): now also D7.1 (A)
- net at MX42.2 (ROW): now also D23.2 (A)
- net at MX57.2 (ROW): now also D31.2 (A)
- net at MX74.2 (ROW): now also D39.2 (A)
- net at MX83.2 (ROW): now also D44.2 (A)
- net at MX14.2 (ROW): now also D8.2 (A)
- net at MX28.2 (ROW): now also D15.1 (A)
- net at MX58.2 (ROW): now also D31.1 (A), MX59.2 (ROW)
- net at MX58.3 (LED), R62.1: now also MX59.3 (LED)
- net at MX75.2 (ROW): now also D39.1 (A)
- net at MX84.2 (ROW): now also D44.1 (A)
- net at MX29.2 (ROW): now also D16.1 (A)
- net at MX44.2 (ROW): now also D24.1 (A)
- net at MX60.2 (ROW): now also D32.1 (A)
- net at MX76.2 (ROW): now also D40.1 (A)
- net at MX85.2 (ROW): now also D45.1 (A)
- net at SW1.S1: now also D8.1 (A)
- new net: MX61.1 (COL), MX62.1 (COL)
- new net: MX61.4 (LEDGND), MX62.4 (LEDGND)
- new net: MX58.1 (COL), MX59.1 (COL)
- new net: MX58.4 (LEDGND), MX59.4 (LEDGND)
- new net: D23.1 (A), MX43.2 (ROW)
Other:
- note removed: "Keyboard Matrix (ISO, 82 key) + LED + Rotary"
- moved on the sheet: C8, C9, MX1, MX10, MX11, MX12, MX13, MX14, MX15, MX16, MX17, MX18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

Commit message: continued routing
Connections:
- net COL0: now also MX1.1 (COL), MX15.1 (COL), MX30.1 (COL), MX45.1 (COL), MX61.1 (COL), MX62.1 (COL), MX77.1 (COL)
- net COL1: now also MX16.1 (COL), MX2.1 (COL), MX63.1 (COL), MX78.1 (COL)
- net COL10: now also MX10.1 (COL), MX25.1 (COL), MX39.1 (COL), MX54.1 (COL), MX72.1 (COL), MX81.1 (COL)
- net COL11: now also MX11.1 (COL), MX26.1 (COL), MX40.1 (COL), MX55.1 (COL), MX73.1 (COL), MX82.1 (COL)
- net COL12: now also MX12.1 (COL), MX27.1 (COL), MX41.1 (COL), MX56.1 (COL)
- net COL13: now also MX13.1 (COL), MX42.1 (COL), MX57.1 (COL), MX74.1 (COL), MX83.1 (COL)
- net COL14: now also MX14.1 (COL), MX28.1 (COL), MX43.1 (COL), MX58.1 (COL), MX59.1 (COL), MX75.1 (COL), MX84.1 (COL)
- net COL15: now also MX29.1 (COL), MX44.1 (COL), MX60.1 (COL), MX76.1 (COL), MX85.1 (COL)
- net COL2: now also MX17.1 (COL), MX3.1 (COL), MX31.1 (COL), MX46.1 (COL), MX64.1 (COL), MX79.1 (COL)
- net COL3: now also MX18.1 (COL), MX32.1 (COL), MX4.1 (COL), MX47.1 (COL), MX65.1 (COL)
- net COL4: now also MX19.1 (COL), MX33.1 (COL), MX48.1 (COL), MX5.1 (COL), MX66.1 (COL)
- net COL5: now also MX20.1 (COL), MX34.1 (COL), MX49.1 (COL), MX67.1 (COL)
- net COL6: now also MX21.1 (COL), MX35.1 (COL), MX50.1 (COL), MX6.1 (COL), MX68.1 (COL), MX80.1 (COL)
- net COL7: now also MX22.1 (COL), MX36.1 (COL), MX51.1 (COL), MX69.1 (COL), MX7.1 (COL)
- net COL8: now also MX23.1 (COL), MX37.1 (COL), MX52.1 (COL), MX70.1 (COL), MX8.1 (COL)
- net COL9: now also MX24.1 (COL), MX38.1 (COL), MX53.1 (COL), MX71.1 (COL), MX9.1 (COL)
- net ROW0: now also D1.3 (K), D2.3 (K), D3.3 (K), D4.3 (K), D5.3 (K), D6.3 (K), D7.3 (K), D8.3 (K)
- net ROW1: now also D10.3 (K), D11.3 (K), D12.3 (K), D13.3 (K), D14.3 (K), D15.3 (K), D16.3 (K), D9.3 (K)
- net ROW2: now also D17.3 (K), D18.3 (K), D19.3 (K), D20.3 (K), D21.3 (K), D22.3 (K), D23.3 (K), D24.3 (K)
- net ROW3: now also D25.3 (K), D26.3 (K), D27.3 (K), D28.3 (K), D29.3 (K), D30.3 (K), D31.3 (K), D32.3 (K)
- net ROW4: now also D33.3 (K), D34.3 (K), D35.3 (K), D36.3 (K), D37.3 (K), D38.3 (K), D39.3 (K), D40.3 (K)
- net ROW5: now also D41.3 (K), D42.3 (K), D43.3 (K), D44.3 (K), D45.3 (K)

Commit message: began renaming project
Parts:
- added R53: 680R, Resistor_SMD:R_0603_1608Metric_Pad1.05x0.95mm_HandSolder, symbol Device:R_Small
- renumbered R5 to R10, R6 to R11, R7 to R12, R8 to R13, R9 to R14, R10 to R15, R11 to R16, R12 to R17, R13 to R18, R14 to R19, R15 to R20, R16 to R21, R17 to R22, R18 to R23, R19 to R24, R20 to R25, R21 to R26, R22 to R27, R23 to R28, R24 to R29, R25 to R30, R26 to R31, R27 to R32, R28 to R33, R29 to R34, R30 to R35, R31 to R36, R32 to R37, R33 to R38, R34 to R39, R35 to R40, R36 to R41, R37 to R42, R38 to R43, R39 to R44, R40 to R45, R41 to R46, R42 to R47, R43 to R48, R44 to R49, R45 to R50, R46 to R51, R47 to R52, R48 to R54, R49 to R55, R50 to R56, R51 to R57, R52 to R58, R53 to R59, R54 to R60, R55 to R61, R56 to R62, R57 to R63, R58 to R64, R59 to R65, R60 to R66, R61 to R67, R62 to R68, R63 to R69, R64 to R70, R65 to R71, R66 to R72, R67 to R73, R68 to R74, R69 to R75, R70 to R76, R71 to R77, R72 to R78, R73 to R79, R74 to R80, R75 to R81, R76 to R82, R77 to R83, R78 to R84, R79 to R85, R80 to R86, R81 to R87, R82 to R88, R83 to R89, R4 to R9, R84 to R90, R85 to R91, R86 to R92, R87 to R93
Connections:
- net +5V: now also R10.2, R11.2, R12.2, R13.2, R14.2, R15.2, R16.2, R17.2, R18.2, R19.2, R20.2, R21.2, R22.2, R23.2, R25.2, R26.2, R27.2, R28.2, R29.2, R30.2, R31.2, R32.2, R33.2, R34.2, R35.2, R36.2, R37.2, R38.2, R39.2, R40.2, R41.2, R42.2, R43.2, R44.2, R45.2, R46.2, R47.2, R48.2, R49.2, R50.2, R51.2, R52.2, R54.2, R55.2, R56.2, R57.2, R58.2, R59.2, R60.2, R61.2, R62.2, R63.2, R64.2, R65.2, R66.2, R67.2, R68.2, R69.2, R70.2, R71.2, R72.2, R73.2, R74.2, R75.2, R76.2, R77.2, R78.2, R79.2, R80.2, R81.2, R82.2, R83.2, R84.2, R85.2, R86.2, R87.2, R88.2, R89.2, R90.2, R91.2, R92.2, R93.2, R53.2
- net LED-: now also MX1.4 (LEDGND), MX10.4 (LEDGND), MX11.4 (LEDGND), MX12.4 (LEDGND), MX13.4 (LEDGND), MX14.4 (LEDGND), MX15.4 (LEDGND), MX16.4 (LEDGND), MX17.4 (LEDGND), MX18.4 (LEDGND), MX19.4 (LEDGND), MX2.4 (LEDGND), MX20.4 (LEDGND), MX21.4 (LEDGND), MX22.4 (LEDGND), MX23.4 (LEDGND), MX24.4 (LEDGND), MX25.4 (LEDGND), MX26.4 (LEDGND), MX27.4 (LEDGND), MX28.4 (LEDGND), MX29.4 (LEDGND), MX3.4 (LEDGND), MX30.4 (LEDGND), MX31.4 (LEDGND), MX32.4 (LEDGND), MX33.4 (LEDGND), MX34.4 (LEDGND), MX35.4 (LEDGND), MX36.4 (LEDGND), MX37.4 (LEDGND), MX38.4 (LEDGND), MX39.4 (LEDGND), MX4.4 (LEDGND), MX40.4 (LEDGND), MX41.4 (LEDGND), MX42.4 (LEDGND), MX43.4 (LEDGND), MX44.4 (LEDGND), MX45.4 (LEDGND), MX46.4 (LEDGND), MX47.4 (LEDGND), MX48.4 (LEDGND), MX49.4 (LEDGND), MX5.4 (LEDGND), MX50.4 (LEDGND), MX51.4 (LEDGND), MX52.4 (LEDGND), MX53.4 (LEDGND), MX54.4 (LEDGND), MX55.4 (LEDGND), MX56.4 (LEDGND), MX57.4 (LEDGND), MX58.4 (LEDGND), MX59.4 (LEDGND), MX6.4 (LEDGND), MX60.4 (LEDGND), MX61.4 (LEDGND), MX62.4 (LEDGND), MX63.4 (LEDGND), MX64.4 (LEDGND), MX65.4 (LEDGND), MX66.4 (LEDGND), MX67.4 (LEDGND), MX68.4 (LEDGND), MX69.4 (LEDGND), MX7.4 (LEDGND), MX70.4 (LEDGND), MX71.4 (LEDGND), MX72.4 (LEDGND), MX73.4 (LEDGND), MX74.4 (LEDGND), MX75.4 (LEDGND), MX76.4 (LEDGND), MX77.4 (LEDGND), MX78.4 (LEDGND), MX79.4 (LEDGND), MX8.4 (LEDGND), MX80.4 (LEDGND), MX81.4 (LEDGND), MX82.4 (LEDGND), MX83.4 (LEDGND), MX84.4 (LEDGND), MX85.4 (LEDGND), MX9.4 (LEDGND)
- net at MX43.3 (LED): now also R53.1
