File: isometria-75-pcb-ml/isometria-75-pcb-ml.sch (KiCad schematic (older format))
At the start: 23 parts, among them J1 USB, J2 SWD, Q1 AO3400A, Q2 AO3401A, Q3 2N7002, U1 TXB0101, U2 XC6206P332MR, U3 nRF52840_holyiot_18010

Commit message: final checks
Parts:
- added C8: 100n, Capacitor_SMD:C_0603_1608Metric_Pad1.05x0.95mm_HandSolder, symbol Device:C_Small
Connections:
- net +3V3: now also C8.1
- net +5V: no longer U3.22 (VBUS)
- net GND: now also C8.2
- net chgsense renamed VBUS
- net VBUS: now also U3.22 (VBUS)
Other:
- moved on the sheet: C3, C4, C5, C6, C7, U2
Changed lines of the file:
@@
 Wire Wire Line
 	1750 1050 1750 900
-Text GLabel 1150 950  2    50   Output ~ 0
-chgsense
 Text GLabel 1150 1250 2    50   BiDi ~ 0
 USB-D+
@@
 L power:+5V #PWR011
 U 1 1 5E6577C1
-P 2100 2550
-F 0 "#PWR011" H 2100 2400 50  0001 C CNN
-F 1 "+5V" H 2200 2650 50  0000 C CNN
-F 2 "" H 2100 2550 50  0001 C CNN
-F 3 "" H 2100 2550 50  0001 C CNN
-	1    2100 2550
-	1    0    0    -1
-$EndComp
-Connection ~ 2650 2850
-Connection ~ 3050 2550
+P 1900 2550
+F 0 "#PWR011" H 1900 2400 50  0001 C CNN
+F 1 "+5V" H 2000 2650 50  0000 C CNN
+F 2 "" H 1900 2550 50  0001 C CNN
+F 3 "" H 1900 2550 50  0001 C CNN
+	1    1900 2550
+	1    0    0    -1
+$EndComp
+Connection ~ 2450 2850
+Connection ~ 2850 2550
 $Comp
 L Device:C_Small C7
 U 1 1 5E6440A6
-P 3050 2700
-F 0 "C7" H 3142 2746 50  0000 L CNN
-F 1 "1uF" H 3142 2655 50  0000 L CNN
-F 2 "Capacitor_SMD:C_0603_1608Metric_Pad1.05x0.95mm_HandSolder" H 3050 2700 50  0001 C CNN
-F 3 "~" H 3050 2700 50  0001 C CNN
-F 4 "C52923" H 3050 2700 50  0001 C CNN "LCSC"
-	1    3050 2700
+P 2850 2700
+F 0 "C7" H 2942 2746 50  0000 L CNN
+F 1 "1uF" H 2942 2655 50  0000 L CNN
+F 2 "Capacitor_SMD:C_0603_1608Metric_Pad1.05x0.95mm_HandSolder" H 2850 2700 50  0001 C CNN
+F 3 "~" H 2850 2700 50  0001 C CNN
+F 4 "C52923" H 2850 2700 50  0001 C CNN "LCSC"
+	1    2850 2700
 	1    0    0    -1
 $EndComp
@@
 L Device:C_Small C6
 U 1 1 5E643787
-P 2100 2700
-F 0 "C6" H 2192 2746 50  0000 L CNN
-F 1 "1uF" H 2192 2655 50  0000 L CNN
-F 2 "Capacitor_SMD:C_0603_1608Metric_Pad1.05x0.95mm_HandSolder" H 2100 2700 50  0001 C CNN
-F 3 "~" H 2100 2700 50  0001 C CNN
-F 4 "C52923" H 2100 2700 50  0001 C CNN "LCSC"
-	1    2100 2700
+P 1900 2700
+F 0 "C6" H 1992 2746 50  0000 L CNN
+F 1 "1uF" H 1992 2655 50  0000 L CNN
+F 2 "Capacitor_SMD:C_0603_1608Metric_Pad1.05x0.95mm_HandSolder" H 1900 2700 50  0001 C CNN
+F 3 "~" H 1900 2700 50  0001 C CNN
+F 4 "C52923" H 1900 2700 50  0001 C CNN "LCSC"
+	1    1900 2700
 	1    0    0    -1
 $EndComp
@@
 L kicad-keyboard-parts:XC6206PxxxMR-Regulator_Linear U2
 U 1 1 5E63D7AB
-P 2650 2550
-F 0 "U2" H 2650 2792 50  0000 C CNN
-F 1 "XC6206P332MR" H 2650 2701 50  0000 C CNN
-F 2 "Package_TO_SOT_SMD:SOT-23" H 2650 2775 50  0001 C CIN
-F 3 "https://www.torexsemi.com/file/xc6206/XC6206.pdf" H 2650 2550 50  0001 C CNN
-F 4 "C5446" H 2650 2550 50  0001 C CNN "LCSC"
-	1    2650 2550
+P 2450 2550
+F 0 "U2" H 2450 2792 50  0000 C CNN
+F 1 "XC6206P332MR" H 2450 2701 50  0000 C CNN
+F 2 "Package_TO_SOT_SMD:SOT-23" H 2450 2775 50  0001 C CIN
+F 3 "https://www.torexsemi.com/file/xc6206/XC6206.pdf" H 2450 2550 50  0001 C CNN
+F 4 "C5446" H 2450 2550 50  0001 C CNN "LCSC"
+	1    2450 2550
 	1    0    0    -1
 $EndComp
@@
 L power:+3.3V #PWR012
 U 1 1 5E625D2A
-P 3050 2550
-F 0 "#PWR012" H 3050 2400 50  0001 C CNN
-F 1 "+3.3V" H 3200 2650 50  0000 C CNN
-F 2 "" H 3050 2550 50  0001 C CNN
-F 3 "" H 3050 2550 50  0001 C CNN
-	1    3050 2550
+P 2850 2550
+F 0 "#PWR012" H 2850 2400 50  0001 C CNN
+F 1 "+3.3V" H 3000 2650 50  0000 C CNN
+F 2 "" H 2850 2550 50  0001 C CNN
+F 3 "" H 2850 2550 50  0001 C CNN
+	1    2850 2550
 	1    0    0    -1
 $EndComp
@@
 	1900 1800 550  1800
 Wire Wire Line
-	1700 2800 1700 2850
-Wire Wire Line
-	2950 2550 3050 2550
-Wire Wire Line
-	1700 2600 1700 2550
-Wire Wire Line
-	3050 2600 3050 2550
-Wire Wire Line
-	3050 2800 3050 2850
+	1500 2800 1500 2850
+Wire Wire Line
+	2750 2550 2850 2550
+Wire Wire Line
+	1500 2600 1500 2550
+Wire Wire Line
+	2850 2600 2850 2550
+Wire Wire Line
+	2850 2800 2850 2850
 Wire Notes Line style solid
 	3500 1800 2000 1800
@@
 L Device:C_Small C5
 U 1 1 5E74EFE9
-P 1700 2700
-F 0 "C5" H 1792 2746 50  0000 L CNN
-F 1 "4.7uF" H 1792 2655 50  0000 L CNN
-F 2 "Capacitor_SMD:C_0603_1608Metric_Pad1.05x0.95mm_HandSolder" H 1700 2700 50  0001 C CNN
-F 3 "~" H 1700 2700 50  0001 C CNN
-F 4 "C23733" H 1700 2700 50  0001 C CNN "LCSC"
-	1    1700 2700
-	1    0    0    -1
-$EndComp
-Connection ~ 1700 2850
-Connection ~ 1700 2550
-Wire Wire Line
-	2100 2600 2100 2550
-Connection ~ 2100 2550
-Wire Wire Line
-	2100 2800 2100 2850
-Connection ~ 2100 2850
-Wire Wire Line
-	2650 2850 3050 2850
-Wire Wire Line
-	2100 2550 2350 2550
-Wire Wire Line
-	2100 2850 2650 2850
-Wire Wire Line
-	1700 2850 2100 2850
-Wire Wire Line
-	1700 2550 2100 2550
+P 1500 2700
+F 0 "C5" H 1592 2746 50  0000 L CNN
+F 1 "4.7uF" H 1592 2655 50  0000 L CNN
+F 2 "Capacitor_SMD:C_0603_1608Metric_Pad1.05x0.95mm_HandSolder" H 1500 2700 50  0001 C CNN
+F 3 "~" H 1500 2700 50  0001 C CNN
+F 4 "C23733" H 1500 2700 50  0001 C CNN "LCSC"
+	1    1500 2700
+	1    0    0    -1
+$EndComp
+Connection ~ 1500 2850
+Connection ~ 1500 2550
+Wire Wire Line
+	1900 2600 1900 2550
+Connection ~ 1900 2550
+Wire Wire Line
+	1900 2800 1900 2850
+Connection ~ 1900 2850
+Wire Wire Line
+	2450 2850 2850 2850
+Wire Wire Line
+	1900 2550 2150 2550
+Wire Wire Line
+	1900 2850 2450 2850
+Wire Wire Line
+	1500 2850 1900 2850
+Wire Wire Line
+	1500 2550 1900 2550
 Text GLabel 2650 5250 0    50   Input ~ 0
 ROTB
 Text GLabel 2650 5150 0    50   Input ~ 0
 ROTA
-Text GLabel 2750 6150 0    50   Input ~ 0
+Text GLabel 2750 6150 0    50   Output ~ 0
 COL15
-Text GLabel 2750 6050 0    50   Input ~ 0
+Text GLabel 2750 6050 0    50   Output ~ 0
 COL14
 Text GLabel 2750 5950 0    50   Output ~ 0
@@
 L Device:C_Small C4
 U 1 1 5E88206E
-P 1300 2700
-F 0 "C4" H 1392 2746 50  0000 L CNN
-F 1 "4.7u" H 1392 2655 50  0000 L CNN
-F 2 "Capacitor_SMD:C_0603_1608Metric_Pad1.05x0.95mm_HandSolder" H 1300 2700 50  0001 C CNN
-F 3 "~" H 1300 2700 50  0001 C CNN
-F 4 "C7171" H 1300 2700 50  0001 C CNN "LCSC"
-	1    1300 2700
+P 1100 2700
+F 0 "C4" H 1192 2746 50  0000 L CNN
+F 1 "4.7u" H 1192 2655 50  0000 L CNN
+F 2 "Capacitor_SMD:C_0603_1608Metric_Pad1.05x0.95mm_HandSolder" H 1100 2700 50  0001 C CNN
+F 3 "~" H 1100 2700 50  0001 C CNN
+F 4 "C7171" H 1100 2700 50  0001 C CNN "LCSC"
+	1    1100 2700
 	1    0    0    -1
 $EndComp
@@
 L Device:C_Small C3
 U 1 1 5E884105
-P 850 2700
-F 0 "C3" H 942 2746 50  0000 L CNN
-F 1 "100uF" H 942 2655 50  0000 L CNN
-F 2 "Capacitor_Tantalum_SMD:CP_EIA-3528-21_Kemet-B" H 850 2700 50  0001 C CNN
-F 3 "~" H 850 2700 50  0001 C CNN
-F 4 "C16133" H 850 2700 50  0001 C CNN "LCSC"
-	1    850  2700
+P 650 2700
+F 0 "C3" H 742 2746 50  0000 L CNN
+F 1 "100uF" H 742 2655 50  0000 L CNN
+F 2 "Capacitor_Tantalum_SMD:CP_EIA-3528-21_Kemet-B" H 650 2700 50  0001 C CNN
+F 3 "~" H 650 2700 50  0001 C CNN
+F 4 "C16133" H 650 2700 50  0001 C CNN "LCSC"
+	1    650  2700
 	1    0    0    -1
 $EndComp
@@
 L power:GND #PWR013
 U 1 1 5E626CC8
-P 2650 2850
-F 0 "#PWR013" H 2650 2600 50  0001 C CNN
-F 1 "GND" H 2655 2677 50  0000 C CNN
-F 2 "" H 2650 2850 50  0001 C CNN
-F 3 "" H 2650 2850 50  0001 C CNN
-	1    2650 2850
-	1    0    0    -1
-$EndComp
-Wire Wire Line
-	1700 2850 1300 2850
-Wire Wire Line
-	1300 2850 1300 2800
-Wire Wire Line
-	1300 2600 1300 2550
-Wire Wire Line
-	1300 2550 1700 2550
+P 2450 2850
+F 0 "#PWR013" H 2450 2600 50  0001 C CNN
+F 1 "GND" H 2455 2677 50  0000 C CNN
+F 2 "" H 2450 2850 50  0001 C CNN
+F 3 "" H 2450 2850 50  0001 C CNN
+	1    2450 2850
+	1    0    0    -1
+$EndComp
+Wire Wire Line
+	1500 2850 1100 2850
+Wire Wire Line
+	1100 2850 1100 2800
+Wire Wire Line
+	1100 2600 1100 2550
+Wire Wire Line
+	1100 2550 1500 2550
 $Comp
 L Device:R_Small R3
@@
 Connection ~ 3000 1550
 Wire Wire Line
-	850  2600 850  2550
-Wire Wire Line
-	850  2550 1300 2550
-Connection ~ 1300 2550
-Wire Wire Line
-	850  2800 850  2850
-Wire Wire Line
-	850  2850 1300 2850
-Connection ~ 1300 2850
+	650  2600 650  2550
+Wire Wire Line
+	650  2550 1100 2550
+Connection ~ 1100 2550
+Wire Wire Line
+	650  2800 650  2850
+Wire Wire Line
+	650  2850 1100 2850
+Connection ~ 1100 2850
 $Comp
 L kicad-keyboard-parts:nRF52840_holyiot_18010 U3
@@
 UG_EN
 $Comp
-L power:+5V #PWR020
-U 1 1 5F9B72BB
-P 3600 7250
-F 0 "#PWR020" H 3600 7100 50  0001 C CNN
-F 1 "+5V" H 3615 7423 50  0000 C CNN
-F 2 "" H 3600 7250 50  0001 C CNN
-F 3 "" H 3600 7250 50  0001 C CNN
-	1    3600 7250
-	1    0    0    -1
-$EndComp
-Wire Wire Line
-	3600 7250 3600 7300
-Wire Wire Line
-	3600 7300 3750 7300
-Wire Wire Line
-	3750 7300 3750 6750
-$Comp
 L Device:R_Small R8
 U 1 1 5F9C1263
@@
 Wire Notes Line style solid
 	3500 2000 3500 3250
+Text GLabel 3750 6900 3    50   Input ~ 0
+VBUS
+Wire Wire Line
+	3750 6900 3750 6750
+$Comp
+L Device:C_Small C8
+U 1 1 5FAA1C6E
+P 3200 2700
+F 0 "C8" H 3292 2746 50  0000 L CNN
+F 1 "100n" H 3292 2655 50  0000 L CNN
+F 2 "Capacitor_SMD:C_0603_1608Metric_Pad1.05x0.95mm_HandSolder" H 3200 2700 50  0001 C CNN
+F 3 "~" H 3200 2700 50  0001 C CNN
+F 4 "C52923" H 3200 2700 50  0001 C CNN "LCSC"
+	1    3200 2700
+	1    0    0    -1
+$EndComp
+Wire Wire Line
+	2850 2850 3200 2850
+Wire Wire Line
+	3200 2850 3200 2800
+Connection ~ 2850 2850
+Wire Wire Line
+	3200 2600 3200 2550
+Wire Wire Line
+	3200 2550 2850 2550
+Text GLabel 1150 950  2    50   Input ~ 0
+VBUS
 $EndSCHEMATC

Commit message: no clue
Parts:
- C1, C2: LCSC (none) -> C386152
- C3: value 100uF -> 100u
- C4: LCSC C7171 -> C1705
- C5: value 4.7uF -> 4.7u; LCSC C23733 -> C1705
- C6, C7: value 1uF -> 1u; LCSC C52923 -> C15849
- C8: LCSC C52923 -> C386152
- J1: LCSC (none) -> C136657
- Q1: LCSC C20917 -> C344010
- Q2: LCSC (none) -> C15127
- Q3: LCSC (none) -> C306856
- R1, R4, R6: LCSC (none) -> C384294
- R2: LCSC C25076 -> C163844
- R3: LCSC C25744 -> C384294
- R5: LCSC (none) -> C163844
- R7: LCSC (none) -> C170462
- R8: LCSC (none) -> C163894
- U2: LCSC C5446 -> C347376
Changed lines of the file:
@@
 F 2 "Package_TO_SOT_SMD:SOT-23" H 3100 1450 50  0001 C CNN
 F 3 "https://datasheet.lcsc.com/szlcsc/Alpha-Omega-Semicon-AOS-AO3400A_C20917.pdf" H 2900 1350 50  0001 C CNN
-F 4 "C20917" H 2900 1350 50  0001 C CNN "LCSC"
+F 4 "C344010" H 2900 1350 50  0001 C CNN "LCSC"
 	1    2900 1350
 	1    0    0    -1
@@
 F 2 "Resistor_SMD:R_0603_1608Metric_Pad1.05x0.95mm_HandSolder" H 2600 1350 50  0001 C CNN
 F 3 "~" H 2600 1350 50  0001 C CNN
-F 4 "C25076" H 2600 1350 50  0001 C CNN "LCSC"
+F 4 "C163844" H 2600 1350 50  0001 C CNN "LCSC"
 	1    2600 1350
 	0    -1   1    0
@@
 F 2 "Connector_JST:JST_SH_SM05B-SRSS-TB_1x05-1MP_P1.00mm_Horizontal" H 950 1150 50  0001 C CNN
 F 3 "http://www.jst-mfg.com/product/pdf/eng/ePH.pdf" H 950 1150 50  0001 C CNN
-F 4 "" H 950 1150 50  0001 C CNN "LCSC"
+F 4 "C136657" H 950 1150 50  0001 C CNN "LCSC"
 	1    950  1150
 	-1   0    0    1
@@
 P 2850 2700
 F 0 "C7" H 2942 2746 50  0000 L CNN
-F 1 "1uF" H 2942 2655 50  0000 L CNN
+F 1 "1u" H 2942 2655 50  0000 L CNN
 F 2 "Capacitor_SMD:C_0603_1608Metric_Pad1.05x0.95mm_HandSolder" H 2850 2700 50  0001 C CNN
 F 3 "~" H 2850 2700 50  0001 C CNN
-F 4 "C52923" H 2850 2700 50  0001 C CNN "LCSC"
+F 4 "C15849" H 2850 2700 50  0001 C CNN "LCSC"
 	1    2850 2700
 	1    0    0    -1
@@
 P 1900 2700
 F 0 "C6" H 1992 2746 50  0000 L CNN
-F 1 "1uF" H 1992 2655 50  0000 L CNN
+F 1 "1u" H 1992 2655 50  0000 L CNN
 F 2 "Capacitor_SMD:C_0603_1608Metric_Pad1.05x0.95mm_HandSolder" H 1900 2700 50  0001 C CNN
 F 3 "~" H 1900 2700 50  0001 C CNN
-F 4 "C52923" H 1900 2700 50  0001 C CNN "LCSC"
+F 4 "C15849" H 1900 2700 50  0001 C CNN "LCSC"
 	1    1900 2700
 	1    0    0    -1
@@
 F 2 "Package_TO_SOT_SMD:SOT-23" H 2450 2775 50  0001 C CIN
 F 3 "https://www.torexsemi.com/file/xc6206/XC6206.pdf" H 2450 2550 50  0001 C CNN
-F 4 "C5446" H 2450 2550 50  0001 C CNN "LCSC"
+F 4 "C347376" H 2450 2550 50  0001 C CNN "LCSC"
 	1    2450 2550
 	1    0    0    -1
@@
 P 1500 2700
 F 0 "C5" H 1592 2746 50  0000 L CNN
-F 1 "4.7uF" H 1592 2655 50  0000 L CNN
+F 1 "4.7u" H 1592 2655 50  0000 L CNN
 F 2 "Capacitor_SMD:C_0603_1608Metric_Pad1.05x0.95mm_HandSolder" H 1500 2700 50  0001 C CNN
 F 3 "~" H 1500 2700 50  0001 C CNN
-F 4 "C23733" H 1500 2700 50  0001 C CNN "LCSC"
+F 4 "C1705" H 1500 2700 50  0001 C CNN "LCSC"
 	1    1500 2700
 	1    0    0    -1
@@
 F 2 "Capacitor_SMD:C_0603_1608Metric_Pad1.05x0.95mm_HandSolder" H 1100 2700 50  0001 C CNN
 F 3 "~" H 1100 2700 50  0001 C CNN
-F 4 "C7171" H 1100 2700 50  0001 C CNN "LCSC"
+F 4 "C1705" H 1100 2700 50  0001 C CNN "LCSC"
 	1    1100 2700
 	1    0    0    -1
@@
 P 650 2700
 F 0 "C3" H 742 2746 50  0000 L CNN
-F 1 "100uF" H 742 2655 50  0000 L CNN
+F 1 "100u" H 742 2655 50  0000 L CNN
 F 2 "Capacitor_Tantalum_SMD:CP_EIA-3528-21_Kemet-B" H 650 2700 50  0001 C CNN
 F 3 "~" H 650 2700 50  0001 C CNN
@@
 F 2 "Resistor_SMD:R_0603_1608Metric_Pad1.05x0.95mm_HandSolder" H 2450 1450 50  0001 C CNN
 F 3 "~" H 2450 1450 50  0001 C CNN
-F 4 "C25744" H 2450 1450 50  0001 C CNN "LCSC"
+F 4 "C384294" H 2450 1450 50  0001 C CNN "LCSC"
 	1    2450 1450
 	1    0    0    -1
@@
 F 2 "Resistor_SMD:R_0603_1608Metric_Pad1.05x0.95mm_HandSolder" H 4200 900 50  0001 C CNN
 F 3 "~" H 4200 900 50  0001 C CNN
+F 4 "C384294" H 4200 900 50  0001 C CNN "LCSC"
 	1    4200 900
 	-1   0    0    1
@@
 F 2 "Capacitor_SMD:C_0603_1608Metric_Pad1.05x0.95mm_HandSolder" H 3900 900 50  0001 C CNN
 F 3 "~" H 3900 900 50  0001 C CNN
+F 4 "C386152" H 3900 900 50  0001 C CNN "LCSC"
 	1    3900 900
 	1    0    0    -1
@@
 F 2 "Capacitor_SMD:C_0603_1608Metric_Pad1.05x0.95mm_HandSolder" H 5250 900 50  0001 C CNN
 F 3 "~" H 5250 900 50  0001 C CNN
+F 4 "C386152" H 5250 900 50  0001 C CNN "LCSC"
 	1    5250 900
 	1    0    0    -1
@@
 F 2 "Package_TO_SOT_SMD:SOT-23" H 4800 2675 50  0001 L CIN
 F 3 "https://www.onsemi.com/pub/Collateral/NDS7002A-D.PDF" H 4600 2750 50  0001 L CNN
+F 4 " C306856" H 4600 2750 50  0001 C CNN "LCSC"
 	1    4600 2750
 	1    0    0    -1
@@
 F 2 "Package_TO_SOT_SMD:SOT-23" H 5100 2325 50  0001 L CIN
 F 3 "http://www.aosmd.com/pdfs/datasheet/AO3401A.pdf" H 4900 2400 50  0001 L CNN
+F 4 " C15127" H 4900 2400 50  0001 C CNN "LCSC"
 	1    4900 2400
 	1    0    0    1
@@
 F 2 "Resistor_SMD:R_0603_1608Metric_Pad1.05x0.95mm_HandSolder" H 4700 2250 50  0001 C CNN
 F 3 "~" H 4700 2250 50  0001 C CNN
+F 4 "C384294" H 4700 2250 50  0001 C CNN "LCSC"
 	1    4700 2250
 	-1   0    0    1
@@
 F 2 "Resistor_SMD:R_0603_1608Metric_Pad1.05x0.95mm_HandSolder" H 4300 2850 50  0001 C CNN
 F 3 "~" H 4300 2850 50  0001 C CNN
+F 4 "C384294" H 4300 2850 50  0001 C CNN "LCSC"
 	1    4300 2850
 	1    0    0    -1
@@
 F 2 "Resistor_SMD:R_0603_1608Metric_Pad1.05x0.95mm_HandSolder" H 4100 2750 50  0001 C CNN
 F 3 "~" H 4100 2750 50  0001 C CNN
+F 4 "C163844" H 4100 2750 50  0001 C CNN "LCSC"
 	1    4100 2750
 	0    1    1    0
@@
 F 2 "Resistor_SMD:R_0603_1608Metric_Pad1.05x0.95mm_HandSolder" H 1850 5650 50  0001 C CNN
 F 3 "~" H 1850 5650 50  0001 C CNN
+F 4 "C163894" H 1850 5650 50  0001 C CNN "LCSC"
 	1    1850 5650
 	1    0    0    -1
@@
 F 2 "Resistor_SMD:R_0603_1608Metric_Pad1.05x0.95mm_HandSolder" H 1850 5450 50  0001 C CNN
 F 3 "~" H 1850 5450 50  0001 C CNN
+F 4 "C170462" H 1850 5450 50  0001 C CNN "LCSC"
 	1    1850 5450
 	1    0    0    -1
@@
 F 2 "Capacitor_SMD:C_0603_1608Metric_Pad1.05x0.95mm_HandSolder" H 3200 2700 50  0001 C CNN
 F 3 "~" H 3200 2700 50  0001 C CNN
-F 4 "C52923" H 3200 2700 50  0001 C CNN "LCSC"
+F 4 "C386152" H 3200 2700 50  0001 C CNN "LCSC"
 	1    3200 2700
 	1    0    0    -1
