File: isometria-75-pcb-ml/matrix.sch (KiCad schematic (older format))
At the start: 218 parts, among them SW1 Rotary_Encoder_Switch

Commit message: final checks
Parts:
- renumbered C9 to C10, C8 to C9
Changed lines of the file:
@@
 LED-
 $Comp
-L power:GND #PWR022
+L power:GND #PWR021
 U 1 1 63289F50
 P 18500 1200
-F 0 "#PWR022" H 18500 950 50  0001 C CNN
+F 0 "#PWR021" H 18500 950 50  0001 C CNN
 F 1 "GND" H 18505 1027 50  0000 C CNN
 F 2 "" H 18500 1200 50  0001 C CNN
@@
 	17750 1300 17800 1300
 $Comp
-L Device:C_Small C9
+L Device:C_Small C10
 U 1 1 6349F64A
 P 17800 1400
-F 0 "C9" H 17650 1300 50  0000 L CNN
+F 0 "C10" H 17650 1300 50  0000 L CNN
 F 1 "100nF" H 17650 1200 50  0000 L CNN
 F 2 "Capacitor_SMD:C_0603_1608Metric_Pad1.05x0.95mm_HandSolder" H 17800 1400 50  0001 C CNN
@@
 Connection ~ 17800 1300
 $Comp
-L Device:C_Small C8
+L Device:C_Small C9
 U 1 1 634A1C5F
 P 17800 1000
-F 0 "C8" H 17650 1100 50  0000 L CNN
+F 0 "C9" H 17650 1100 50  0000 L CNN
 F 1 "100nF" H 17650 1200 50  0000 L CNN
 F 2 "Capacitor_SMD:C_0603_1608Metric_Pad1.05x0.95mm_HandSolder" H 17800 1000 50  0001 C CNN
@@
 	17950 800  17950 900
 $Comp
-L power:+3.3V #PWR021
+L power:+3.3V #PWR020
 U 1 1 637D2133
 P 18650 800
-F 0 "#PWR021" H 18650 650 50  0001 C CNN
+F 0 "#PWR020" H 18650 650 50  0001 C CNN
 F 1 "+3.3V" H 18665 973 50  0000 C CNN
 F 2 "" H 18650 800 50  0001 C CNN

Commit message: removed silkscreen labels from obvious components
Parts:
- D1, D10, D11, D12, D13, D14, D15, D16, D17, D18, D19, D2, D20, D21, D22, D23, D24, D25, D26, D27, D28, D29, D3, D30, D31, D32, D33, D34, D35, D36, D37, D38, D39, D4, D40, D41, D42, D43, D44, D45, D5, D6, D7, D8, D9: footprint Package_TO_SOT_SMD:SOT-23 -> kicad-keyboard-parts:SOT-23_stealth
- R10, R11, R12, R13, R14, R15, R16, R17, R18, R19, R20, R21, R22, R23, R25, R26, R27, R28, R29, R30, R31, R32, R33, R34, R35, R36, R37, R38, R39, R40, R41, R42, R43, R44, R45, R46, R47, R48, R49, R50, R51, R52, R53, R54, R55, R56, R57, R58, R59, R60, R61, R62, R63, R64, R65, R66, R67, R68, R69, R70, R71, R72, R73, R74, R75, R76, R77, R78, R79, R80, R81, R82, R83, R84, R85, R86, R87, R88, R89, R90, R91, R92, R93: footprint Resistor_SMD:R_0603_1608Metric_Pad1.05x0.95mm_HandSolder -> kicad-keyboard-parts:R_0603_1608Metric_stealth_HandSolder

Commit message: no clue
Parts:
- C10, C9: value 100nF -> 100n; LCSC C1525 -> C386152
- D1, D10, D11, D12, D13, D14, D15, D16, D17, D18, D19, D2, D20, D21, D22, D23, D24, D25, D26, D27, D28, D29, D3, D30, D31, D32, D33, D34, D35, D36, D37, D38, D39, D4, D40, D41, D42, D43, D44, D45, D5, D6, D7, D8, D9: LCSC (none) -> C727123
- R24, R9: LCSC C25744 -> C384294
