File: isometria-75-pcb-ml/underglow.sch (KiCad schematic (older format))
At the start: 36 parts

Commit message: final checks
Parts:
- renumbered C10 to C11, C11 to C12, C12 to C13, C13 to C14, C14 to C15, C15 to C16, C16 to C17, C17 to C18, C18 to C19, C19 to C20, C20 to C21, C21 to C22, C22 to C23, C23 to C24, C24 to C25, C25 to C26, C26 to C27, C27 to C28
Changed lines of the file:
@@
 P 3000 1650
 AR Path="/5E6E4592" Ref="C?"  Part="1"
-AR Path="/5E6E13F7/5E6E4592" Ref="C10"  Part="1"
-F 0 "C10" H 3092 1696 50  0000 L CNN
+AR Path="/5E6E13F7/5E6E4592" Ref="C11"  Part="1"
+F 0 "C11" H 3092 1696 50  0000 L CNN
 F 1 "100nF" H 3092 1605 50  0000 L CNN
 F 2 "Capacitor_SMD:C_0603_1608Metric_Pad1.05x0.95mm_HandSolder" H 3000 1650 50  0001 C CNN
@@
 P 3850 1650
 AR Path="/5E6FDF24" Ref="C?"  Part="1"
-AR Path="/5E6E13F7/5E6FDF24" Ref="C11"  Part="1"
-F 0 "C11" H 3942 1696 50  0000 L CNN
+AR Path="/5E6E13F7/5E6FDF24" Ref="C12"  Part="1"
+F 0 "C12" H 3942 1696 50  0000 L CNN
 F 1 "100nF" H 3942 1605 50  0000 L CNN
 F 2 "Capacitor_SMD:C_0603_1608Metric_Pad1.05x0.95mm_HandSolder" H 3850 1650 50  0001 C CNN
@@
 P 4700 1650
 AR Path="/5E704C33" Ref="C?"  Part="1"
-AR Path="/5E6E13F7/5E704C33" Ref="C12"  Part="1"
-F 0 "C12" H 4792 1696 50  0000 L CNN
+AR Path="/5E6E13F7/5E704C33" Ref="C13"  Part="1"
+F 0 "C13" H 4792 1696 50  0000 L CNN
 F 1 "100nF" H 4792 1605 50  0000 L CNN
 F 2 "Capacitor_SMD:C_0603_1608Metric_Pad1.05x0.95mm_HandSolder" H 4700 1650 50  0001 C CNN
@@
 P 5550 1650
 AR Path="/5E704C42" Ref="C?"  Part="1"
-AR Path="/5E6E13F7/5E704C42" Ref="C13"  Part="1"
-F 0 "C13" H 5642 1696 50  0000 L CNN
+AR Path="/5E6E13F7/5E704C42" Ref="C14"  Part="1"
+F 0 "C14" H 5642 1696 50  0000 L CNN
 F 1 "100nF" H 5642 1605 50  0000 L CNN
 F 2 "Capacitor_SMD:C_0603_1608Metric_Pad1.05x0.95mm_HandSolder" H 5550 1650 50  0001 C CNN
@@
 P 7200 1650
 AR Path="/5E710C99" Ref="C?"  Part="1"
-AR Path="/5E6E13F7/5E710C99" Ref="C15"  Part="1"
-F 0 "C15" H 7292 1696 50  0000 L CNN
+AR Path="/5E6E13F7/5E710C99" Ref="C16"  Part="1"
+F 0 "C16" H 7292 1696 50  0000 L CNN
 F 1 "100nF" H 7292 1605 50  0000 L CNN
 F 2 "Capacitor_SMD:C_0603_1608Metric_Pad1.05x0.95mm_HandSolder" H 7200 1650 50  0001 C CNN
@@
 P 8050 1650
 AR Path="/5E710CA8" Ref="C?"  Part="1"
-AR Path="/5E6E13F7/5E710CA8" Ref="C16"  Part="1"
-F 0 "C16" H 8142 1696 50  0000 L CNN
+AR Path="/5E6E13F7/5E710CA8" Ref="C17"  Part="1"
+F 0 "C17" H 8142 1696 50  0000 L CNN
 F 1 "100nF" H 8142 1605 50  0000 L CNN
 F 2 "Capacitor_SMD:C_0603_1608Metric_Pad1.05x0.95mm_HandSolder" H 8050 1650 50  0001 C CNN
@@
 P 8900 1650
 AR Path="/5E710CB7" Ref="C?"  Part="1"
-AR Path="/5E6E13F7/5E710CB7" Ref="C17"  Part="1"
-F 0 "C17" H 8992 1696 50  0000 L CNN
+AR Path="/5E6E13F7/5E710CB7" Ref="C18"  Part="1"
+F 0 "C18" H 8992 1696 50  0000 L CNN
 F 1 "100nF" H 8992 1605 50  0000 L CNN
 F 2 "Capacitor_SMD:C_0603_1608Metric_Pad1.05x0.95mm_HandSolder" H 8900 1650 50  0001 C CNN
@@
 P 9750 1650
 AR Path="/5E710CC6" Ref="C?"  Part="1"
-AR Path="/5E6E13F7/5E710CC6" Ref="C18"  Part="1"
-F 0 "C18" H 9842 1696 50  0000 L CNN
+AR Path="/5E6E13F7/5E710CC6" Ref="C19"  Part="1"
+F 0 "C19" H 9842 1696 50  0000 L CNN
 F 1 "100nF" H 9842 1605 50  0000 L CNN
 F 2 "Capacitor_SMD:C_0603_1608Metric_Pad1.05x0.95mm_HandSolder" H 9750 1650 50  0001 C CNN
@@
 P 3000 2800
 AR Path="/5E714331" Ref="C?"  Part="1"
-AR Path="/5E6E13F7/5E714331" Ref="C19"  Part="1"
-F 0 "C19" H 3092 2846 50  0000 L CNN
+AR Path="/5E6E13F7/5E714331" Ref="C20"  Part="1"
+F 0 "C20" H 3092 2846 50  0000 L CNN
 F 1 "100nF" H 3092 2755 50  0000 L CNN
 F 2 "Capacitor_SMD:C_0603_1608Metric_Pad1.05x0.95mm_HandSolder" H 3000 2800 50  0001 C CNN
@@
 P 3850 2800
 AR Path="/5E714340" Ref="C?"  Part="1"
-AR Path="/5E6E13F7/5E714340" Ref="C20"  Part="1"
-F 0 "C20" H 3942 2846 50  0000 L CNN
+AR Path="/5E6E13F7/5E714340" Ref="C21"  Part="1"
+F 0 "C21" H 3942 2846 50  0000 L CNN
 F 1 "100nF" H 3942 2755 50  0000 L CNN
 F 2 "Capacitor_SMD:C_0603_1608Metric_Pad1.05x0.95mm_HandSolder" H 3850 2800 50  0001 C CNN
@@
 	2950 2600 3200 2600
 $Comp
-L power:GND #PWR023
+L power:GND #PWR022
 U 1 1 5E718AF7
 P 2650 1750
-F 0 "#PWR023" H 2650 1500 50  0001 C CNN
+F 0 "#PWR022" H 2650 1500 50  0001 C CNN
 F 1 "GND" H 2655 1577 50  0000 C CNN
 F 2 "" H 2650 1750 50  0001 C CNN
@@
 P 4700 2800
 AR Path="/5E7ECFEE" Ref="C?"  Part="1"
-AR Path="/5E6E13F7/5E7ECFEE" Ref="C21"  Part="1"
-F 0 "C21" H 4792 2846 50  0000 L CNN
+AR Path="/5E6E13F7/5E7ECFEE" Ref="C22"  Part="1"
+F 0 "C22" H 4792 2846 50  0000 L CNN
 F 1 "100nF" H 4792 2755 50  0000 L CNN
 F 2 "Capacitor_SMD:C_0603_1608Metric_Pad1.05x0.95mm_HandSolder" H 4700 2800 50  0001 C CNN
@@
 P 5550 2800
 AR Path="/5E7ECFFD" Ref="C?"  Part="1"
-AR Path="/5E6E13F7/5E7ECFFD" Ref="C22"  Part="1"
-F 0 "C22" H 5642 2846 50  0000 L CNN
+AR Path="/5E6E13F7/5E7ECFFD" Ref="C23"  Part="1"
+F 0 "C23" H 5642 2846 50  0000 L CNN
 F 1 "100nF" H 5642 2755 50  0000 L CNN
 F 2 "Capacitor_SMD:C_0603_1608Metric_Pad1.05x0.95mm_HandSolder" H 5550 2800 50  0001 C CNN
@@
 P 6400 2800
 AR Path="/5E7FCA18" Ref="C?"  Part="1"
-AR Path="/5E6E13F7/5E7FCA18" Ref="C23"  Part="1"
-F 0 "C23" H 6492 2846 50  0000 L CNN
+AR Path="/5E6E13F7/5E7FCA18" Ref="C24"  Part="1"
+F 0 "C24" H 6492 2846 50  0000 L CNN
 F 1 "100nF" H 6492 2755 50  0000 L CNN
 F 2 "Capacitor_SMD:C_0603_1608Metric_Pad1.05x0.95mm_HandSolder" H 6400 2800 50  0001 C CNN
@@
 P 7250 2800
 AR Path="/5E7FCA27" Ref="C?"  Part="1"
-AR Path="/5E6E13F7/5E7FCA27" Ref="C24"  Part="1"
-F 0 "C24" H 7342 2846 50  0000 L CNN
+AR Path="/5E6E13F7/5E7FCA27" Ref="C25"  Part="1"
+F 0 "C25" H 7342 2846 50  0000 L CNN
 F 1 "100nF" H 7342 2755 50  0000 L CNN
 F 2 "Capacitor_SMD:C_0603_1608Metric_Pad1.05x0.95mm_HandSolder" H 7250 2800 50  0001 C CNN
@@
 P 8100 2800
 AR Path="/5E7FCA37" Ref="C?"  Part="1"
-AR Path="/5E6E13F7/5E7FCA37" Ref="C25"  Part="1"
-F 0 "C25" H 8192 2846 50  0000 L CNN
+AR Path="/5E6E13F7/5E7FCA37" Ref="C26"  Part="1"
+F 0 "C26" H 8192 2846 50  0000 L CNN
 F 1 "100nF" H 8192 2755 50  0000 L CNN
 F 2 "Capacitor_SMD:C_0603_1608Metric_Pad1.05x0.95mm_HandSolder" H 8100 2800 50  0001 C CNN
@@
 P 8950 2800
 AR Path="/5E7FCA46" Ref="C?"  Part="1"
-AR Path="/5E6E13F7/5E7FCA46" Ref="C26"  Part="1"
-F 0 "C26" H 9042 2846 50  0000 L CNN
+AR Path="/5E6E13F7/5E7FCA46" Ref="C27"  Part="1"
+F 0 "C27" H 9042 2846 50  0000 L CNN
 F 1 "100nF" H 9042 2755 50  0000 L CNN
 F 2 "Capacitor_SMD:C_0603_1608Metric_Pad1.05x0.95mm_HandSolder" H 8950 2800 50  0001 C CNN
@@
 P 6400 1650
 AR Path="/5E8DE968" Ref="C?"  Part="1"
-AR Path="/5E6E13F7/5E8DE968" Ref="C14"  Part="1"
-F 0 "C14" H 6492 1696 50  0000 L CNN
+AR Path="/5E6E13F7/5E8DE968" Ref="C15"  Part="1"
+F 0 "C15" H 6492 1696 50  0000 L CNN
 F 1 "100nF" H 6492 1605 50  0000 L CNN
 F 2 "Capacitor_SMD:C_0603_1608Metric_Pad1.05x0.95mm_HandSolder" H 6400 1650 50  0001 C CNN
@@
 P 9750 2800
 AR Path="/5F996F0C" Ref="C?"  Part="1"
-AR Path="/5E6E13F7/5F996F0C" Ref="C27"  Part="1"
-F 0 "C27" H 9842 2846 50  0000 L CNN
+AR Path="/5E6E13F7/5F996F0C" Ref="C28"  Part="1"
+F 0 "C28" H 9842 2846 50  0000 L CNN
 F 1 "100nF" H 9842 2755 50  0000 L CNN
 F 2 "Capacitor_SMD:C_0603_1608Metric_Pad1.05x0.95mm_HandSolder" H 9750 2800 50  0001 C CNN

Commit message: no clue
Parts:
- C11, C12, C13, C14, C15, C16, C17, C18, C19, C20, C21, C22, C23, C24, C25, C26, C27, C28: value 100nF -> 100n; LCSC C1525 -> C386152
Changed lines of the file:
@@
 AR Path="/5E6E13F7/5E6E4592" Ref="C11"  Part="1"
 F 0 "C11" H 3092 1696 50  0000 L CNN
-F 1 "100nF" H 3092 1605 50  0000 L CNN
+F 1 "100n" H 3092 1605 50  0000 L CNN
 F 2 "Capacitor_SMD:C_0603_1608Metric_Pad1.05x0.95mm_HandSolder" H 3000 1650 50  0001 C CNN
 F 3 "~" H 3000 1650 50  0001 C CNN
-F 4 "C1525" H 3000 1650 50  0001 C CNN "LCSC"
+F 4 "C386152" H 3000 1650 50  0001 C CNN "LCSC"
 	1    3000 1650
 	1    0    0    -1
@@
 AR Path="/5E6E13F7/5E6FDF24" Ref="C12"  Part="1"
 F 0 "C12" H 3942 1696 50  0000 L CNN
-F 1 "100nF" H 3942 1605 50  0000 L CNN
+F 1 "100n" H 3942 1605 50  0000 L CNN
 F 2 "Capacitor_SMD:C_0603_1608Metric_Pad1.05x0.95mm_HandSolder" H 3850 1650 50  0001 C CNN
 F 3 "~" H 3850 1650 50  0001 C CNN
-F 4 "C1525" H 3850 1650 50  0001 C CNN "LCSC"
+F 4 "C386152" H 3850 1650 50  0001 C CNN "LCSC"
 	1    3850 1650
 	1    0    0    -1
@@
 AR Path="/5E6E13F7/5E704C33" Ref="C13"  Part="1"
 F 0 "C13" H 4792 1696 50  0000 L CNN
-F 1 "100nF" H 4792 1605 50  0000 L CNN
+F 1 "100n" H 4792 1605 50  0000 L CNN
 F 2 "Capacitor_SMD:C_0603_1608Metric_Pad1.05x0.95mm_HandSolder" H 4700 1650 50  0001 C CNN
 F 3 "~" H 4700 1650 50  0001 C CNN
-F 4 "C1525" H 4700 1650 50  0001 C CNN "LCSC"
+F 4 "C386152" H 4700 1650 50  0001 C CNN "LCSC"
 	1    4700 1650
 	1    0    0    -1
@@
 AR Path="/5E6E13F7/5E704C42" Ref="C14"  Part="1"
 F 0 "C14" H 5642 1696 50  0000 L CNN
-F 1 "100nF" H 5642 1605 50  0000 L CNN
+F 1 "100n" H 5642 1605 50  0000 L CNN
 F 2 "Capacitor_SMD:C_0603_1608Metric_Pad1.05x0.95mm_HandSolder" H 5550 1650 50  0001 C CNN
 F 3 "~" H 5550 1650 50  0001 C CNN
-F 4 "C1525" H 5550 1650 50  0001 C CNN "LCSC"
+F 4 "C386152" H 5550 1650 50  0001 C CNN "LCSC"
 	1    5550 1650
 	1    0    0    -1
@@
 AR Path="/5E6E13F7/5E710C99" Ref="C16"  Part="1"
 F 0 "C16" H 7292 1696 50  0000 L CNN
-F 1 "100nF" H 7292 1605 50  0000 L CNN
+F 1 "100n" H 7292 1605 50  0000 L CNN
 F 2 "Capacitor_SMD:C_0603_1608Metric_Pad1.05x0.95mm_HandSolder" H 7200 1650 50  0001 C CNN
 F 3 "~" H 7200 1650 50  0001 C CNN
-F 4 "C1525" H 7200 1650 50  0001 C CNN "LCSC"
+F 4 "C386152" H 7200 1650 50  0001 C CNN "LCSC"
 	1    7200 1650
 	1    0    0    -1
@@
 AR Path="/5E6E13F7/5E710CA8" Ref="C17"  Part="1"
 F 0 "C17" H 8142 1696 50  0000 L CNN
-F 1 "100nF" H 8142 1605 50  0000 L CNN
+F 1 "100n" H 8142 1605 50  0000 L CNN
 F 2 "Capacitor_SMD:C_0603_1608Metric_Pad1.05x0.95mm_HandSolder" H 8050 1650 50  0001 C CNN
 F 3 "~" H 8050 1650 50  0001 C CNN
-F 4 "C1525" H 8050 1650 50  0001 C CNN "LCSC"
+F 4 "C386152" H 8050 1650 50  0001 C CNN "LCSC"
 	1    8050 1650
 	1    0    0    -1
@@
 AR Path="/5E6E13F7/5E710CB7" Ref="C18"  Part="1"
 F 0 "C18" H 8992 1696 50  0000 L CNN
-F 1 "100nF" H 8992 1605 50  0000 L CNN
+F 1 "100n" H 8992 1605 50  0000 L CNN
 F 2 "Capacitor_SMD:C_0603_1608Metric_Pad1.05x0.95mm_HandSolder" H 8900 1650 50  0001 C CNN
 F 3 "~" H 8900 1650 50  0001 C CNN
-F 4 "C1525" H 8900 1650 50  0001 C CNN "LCSC"
+F 4 "C386152" H 8900 1650 50  0001 C CNN "LCSC"
 	1    8900 1650
 	1    0    0    -1
@@
 AR Path="/5E6E13F7/5E710CC6" Ref="C19"  Part="1"
 F 0 "C19" H 9842 1696 50  0000 L CNN
-F 1 "100nF" H 9842 1605 50  0000 L CNN
+F 1 "100n" H 9842 1605 50  0000 L CNN
 F 2 "Capacitor_SMD:C_0603_1608Metric_Pad1.05x0.95mm_HandSolder" H 9750 1650 50  0001 C CNN
 F 3 "~" H 9750 1650 50  0001 C CNN
-F 4 "C1525" H 9750 1650 50  0001 C CNN "LCSC"
+F 4 "C386152" H 9750 1650 50  0001 C CNN "LCSC"
 	1    9750 1650
 	1    0    0    -1
@@
 AR Path="/5E6E13F7/5E714331" Ref="C20"  Part="1"
 F 0 "C20" H 3092 2846 50  0000 L CNN
-F 1 "100nF" H 3092 2755 50  0000 L CNN
+F 1 "100n" H 3092 2755 50  0000 L CNN
 F 2 "Capacitor_SMD:C_0603_1608Metric_Pad1.05x0.95mm_HandSolder" H 3000 2800 50  0001 C CNN
 F 3 "~" H 3000 2800 50  0001 C CNN
-F 4 "C1525" H 3000 2800 50  0001 C CNN "LCSC"
+F 4 "C386152" H 3000 2800 50  0001 C CNN "LCSC"
 	1    3000 2800
 	1    0    0    -1
@@
 AR Path="/5E6E13F7/5E714340" Ref="C21"  Part="1"
 F 0 "C21" H 3942 2846 50  0000 L CNN
-F 1 "100nF" H 3942 2755 50  0000 L CNN
+F 1 "100n" H 3942 2755 50  0000 L CNN
 F 2 "Capacitor_SMD:C_0603_1608Metric_Pad1.05x0.95mm_HandSolder" H 3850 2800 50  0001 C CNN
 F 3 "~" H 3850 2800 50  0001 C CNN
-F 4 "C1525" H 3850 2800 50  0001 C CNN "LCSC"
+F 4 "C386152" H 3850 2800 50  0001 C CNN "LCSC"
 	1    3850 2800
 	1    0    0    -1
@@
 AR Path="/5E6E13F7/5E7ECFEE" Ref="C22"  Part="1"
 F 0 "C22" H 4792 2846 50  0000 L CNN
-F 1 "100nF" H 4792 2755 50  0000 L CNN
+F 1 "100n" H 4792 2755 50  0000 L CNN
 F 2 "Capacitor_SMD:C_0603_1608Metric_Pad1.05x0.95mm_HandSolder" H 4700 2800 50  0001 C CNN
 F 3 "~" H 4700 2800 50  0001 C CNN
-F 4 "C1525" H 4700 2800 50  0001 C CNN "LCSC"
+F 4 "C386152" H 4700 2800 50  0001 C CNN "LCSC"
 	1    4700 2800
 	1    0    0    -1
@@
 AR Path="/5E6E13F7/5E7ECFFD" Ref="C23"  Part="1"
 F 0 "C23" H 5642 2846 50  0000 L CNN
-F 1 "100nF" H 5642 2755 50  0000 L CNN
+F 1 "100n" H 5642 2755 50  0000 L CNN
 F 2 "Capacitor_SMD:C_0603_1608Metric_Pad1.05x0.95mm_HandSolder" H 5550 2800 50  0001 C CNN
 F 3 "~" H 5550 2800 50  0001 C CNN
-F 4 "C1525" H 5550 2800 50  0001 C CNN "LCSC"
+F 4 "C386152" H 5550 2800 50  0001 C CNN "LCSC"
 	1    5550 2800
 	1    0    0    -1
@@
 AR Path="/5E6E13F7/5E7FCA18" Ref="C24"  Part="1"
 F 0 "C24" H 6492 2846 50  0000 L CNN
-F 1 "100nF" H 6492 2755 50  0000 L CNN
+F 1 "100n" H 6492 2755 50  0000 L CNN
 F 2 "Capacitor_SMD:C_0603_1608Metric_Pad1.05x0.95mm_HandSolder" H 6400 2800 50  0001 C CNN
 F 3 "~" H 6400 2800 50  0001 C CNN
-F 4 "C1525" H 6400 2800 50  0001 C CNN "LCSC"
+F 4 "C386152" H 6400 2800 50  0001 C CNN "LCSC"
 	1    6400 2800
 	1    0    0    -1
@@
 AR Path="/5E6E13F7/5E7FCA27" Ref="C25"  Part="1"
 F 0 "C25" H 7342 2846 50  0000 L CNN
-F 1 "100nF" H 7342 2755 50  0000 L CNN
+F 1 "100n" H 7342 2755 50  0000 L CNN
 F 2 "Capacitor_SMD:C_0603_1608Metric_Pad1.05x0.95mm_HandSolder" H 7250 2800 50  0001 C CNN
 F 3 "~" H 7250 2800 50  0001 C CNN
-F 4 "C1525" H 7250 2800 50  0001 C CNN "LCSC"
+F 4 "C386152" H 7250 2800 50  0001 C CNN "LCSC"
 	1    7250 2800
 	1    0    0    -1
@@
 AR Path="/5E6E13F7/5E7FCA37" Ref="C26"  Part="1"
 F 0 "C26" H 8192 2846 50  0000 L CNN
-F 1 "100nF" H 8192 2755 50  0000 L CNN
+F 1 "100n" H 8192 2755 50  0000 L CNN
 F 2 "Capacitor_SMD:C_0603_1608Metric_Pad1.05x0.95mm_HandSolder" H 8100 2800 50  0001 C CNN
 F 3 "~" H 8100 2800 50  0001 C CNN
-F 4 "C1525" H 8100 2800 50  0001 C CNN "LCSC"
+F 4 "C386152" H 8100 2800 50  0001 C CNN "LCSC"
 	1    8100 2800
 	1    0    0    -1
@@
 AR Path="/5E6E13F7/5E7FCA46" Ref="C27"  Part="1"
 F 0 "C27" H 9042 2846 50  0000 L CNN
-F 1 "100nF" H 9042 2755 50  0000 L CNN
+F 1 "100n" H 9042 2755 50  0000 L CNN
 F 2 "Capacitor_SMD:C_0603_1608Metric_Pad1.05x0.95mm_HandSolder" H 8950 2800 50  0001 C CNN
 F 3 "~" H 8950 2800 50  0001 C CNN
-F 4 "C1525" H 8950 2800 50  0001 C CNN "LCSC"
+F 4 "C386152" H 8950 2800 50  0001 C CNN "LCSC"
 	1    8950 2800
 	1    0    0    -1
@@
 AR Path="/5E6E13F7/5E8DE968" Ref="C15"  Part="1"
 F 0 "C15" H 6492 1696 50  0000 L CNN
-F 1 "100nF" H 6492 1605 50  0000 L CNN
+F 1 "100n" H 6492 1605 50  0000 L CNN
 F 2 "Capacitor_SMD:C_0603_1608Metric_Pad1.05x0.95mm_HandSolder" H 6400 1650 50  0001 C CNN
 F 3 "~" H 6400 1650 50  0001 C CNN
-F 4 "C1525" H 6400 1650 50  0001 C CNN "LCSC"
+F 4 "C386152" H 6400 1650 50  0001 C CNN "LCSC"
 	1    6400 1650
 	1    0    0    -1
@@
 AR Path="/5E6E13F7/5F996F0C" Ref="C28"  Part="1"
 F 0 "C28" H 9842 2846 50  0000 L CNN
-F 1 "100nF" H 9842 2755 50  0000 L CNN
+F 1 "100n" H 9842 2755 50  0000 L CNN
 F 2 "Capacitor_SMD:C_0603_1608Metric_Pad1.05x0.95mm_HandSolder" H 9750 2800 50  0001 C CNN
 F 3 "~" H 9750 2800 50  0001 C CNN
-F 4 "C1525" H 9750 2800 50  0001 C CNN "LCSC"
+F 4 "C386152" H 9750 2800 50  0001 C CNN "LCSC"
 	1    9750 2800
 	1    0    0    -1
